Commit message: Refactor launch and configuration files for mobile manipulator; update parameters, enhance controller functionality, and adjust URDF definitions for improved integration.

File: MOBILE_MANIPULATOR/mobile_manipulator_description/urdf/linear_guide.xacro (robot description, xacro)
@@ -6,5 +6,5 @@
         <box size="0.1 0.1 1.0"/>
       </geometry>
-      <origin xyz="0 0 0.5" rpy="0 0 0"/>
+      <origin xyz="0 -0.1 0.5" rpy="0 0 0"/>
       <material name="grey">
         <color rgba="0.5 0.5 0.5 1.0"/>
@@ -15,5 +15,5 @@
         <box size="0.1 0.1 1.0"/>
       </geometry>
-      <origin xyz="0 0 0.5" rpy="0 0 0"/>
+      <origin xyz="0 -0.1 0.5" rpy="0 0 0"/>
     </collision>
     <inertial>
@@ -25,5 +25,5 @@
     <visual>
       <geometry>
-        <box size="0.6 0.6 0.1"/>
+        <box size="0.3 0.3 0.05"/>
       </geometry>
       <origin xyz="0 -0.25 0.05" rpy="0 0 0"/>
@@ -34,5 +34,5 @@
     <collision>
       <geometry>
-        <box size="0.6 0.6 0.1"/>
+        <box size="0.3 0.3 0.05"/>
       </geometry>
       <origin xyz="0 -0.25 0.05" rpy="0 0 0"/>

File: MOBILE_MANIPULATOR/mobile_manipulator_description/urdf/mobile_manipulator.urdf.xacro (robot description, xacro)
@@ -13,5 +13,5 @@
     <parent link="slider"/>
     <child  link="base_link"/>
-    <origin xyz="0 -0.25 0.13" rpy="0 0 0"/>
+    <origin xyz="0 -0.25 0.06" rpy="0 0 0"/>
   </joint>
 <!--

File: MOBILE_MANIPULATOR/mobile_manipulator_description/urdf/mobile_manipulator_ros_contol.xacro (robot description, xacro)
@@ -1,4 +1,5 @@
 <?xml version="1.0"?>
 <robot name="mobile_manipulator" xmlns:xacro="http://www.ros.org/wiki/xacro">
+  <!-- ros2_control setup -->
   <ros2_control name="GazeboSystem" type="system">
     <hardware>
@@ -48,3 +49,84 @@
     </joint>
   </ros2_control>
+  <!-- Transmissions for each controllable joint -->
+  <transmission name="slider_trans">
+    <type>transmission_interface/SimpleTransmission</type>
+    <joint name="slider_joint">
+      <hardwareInterface>hardware_interface/PositionJointInterface</hardwareInterface>
+    </joint>
+    <actuator name="slider_motor">
+      <hardwareInterface>hardware_interface/PositionJointInterface</hardwareInterface>
+      <mechanicalReduction>1</mechanicalReduction>
+    </actuator>
+  </transmission>
+  <transmission name="joint1_trans">
+    <type>transmission_interface/SimpleTransmission</type>
+    <joint name="joint1">
+      <hardwareInterface>hardware_interface/PositionJointInterface</hardwareInterface>
+    </joint>
+    <actuator name="joint1_motor">
+      <hardwareInterface>hardware_interface/PositionJointInterface</hardwareInterface>
+      <mechanicalReduction>1</mechanicalReduction>
+    </actuator>
+  </transmission>
+  <transmission name="joint2_trans">
+    <type>transmission_interface/SimpleTransmission</type>
+    <joint name="joint2">
+      <hardwareInterface>hardware_interface/PositionJointInterface</hardwareInterface>
+    </joint>
+    <actuator name="joint2_motor">
+      <hardwareInterface>hardware_interface/PositionJointInterface</hardwareInterface>
+      <mechanicalReduction>1</mechanicalReduction>
+    </actuator>
+  </transmission>
+  <transmission name="joint3_trans">
+    <type>transmission_interface/SimpleTransmission</type>
+    <joint name="joint3">
+      <hardwareInterface>hardware_interface/PositionJointInterface</hardwareInterface>
+    </joint>
+    <actuator name="joint3_motor">
+      <hardwareInterface>hardware_interface/PositionJointInterface</hardwareInterface>
+      <mechanicalReduction>1</mechanicalReduction>
+    </actuator>
+  </transmission>
+  <transmission name="joint4_trans">
+    <type>transmission_interface/SimpleTransmission</type>
+    <joint name="joint4">
+      <hardwareInterface>hardware_interface/PositionJointInterface</hardwareInterface>
+    </joint>
+    <actuator name="joint4_motor">
+      <hardwareInterface>hardware_interface/PositionJointInterface</hardwareInterface>
+      <mechanicalReduction>1</mechanicalReduction>
+    </actuator>
+  </transmission>
+  <transmission name="joint5_trans">
+    <type>transmission_interface/SimpleTransmission</type>
+    <joint name="joint5">
+      <hardwareInterface>hardware_interface/PositionJointInterface</hardwareInterface>
+    </joint>
+    <actuator name="joint5_motor">
+      <hardwareInterface>hardware_interface/PositionJointInterface</hardwareInterface>
+      <mechanicalReduction>1</mechanicalReduction>
+    </actuator>
+  </transmission>
+  <transmission name="joint6_trans">
+    <type>transmission_interface/SimpleTransmission</type>
+    <joint name="joint6">
+      <hardwareInterface>hardware_interface/PositionJointInterface</hardwareInterface>
+    </joint>
+    <actuator name="joint6_motor">
+      <hardwareInterface>hardware_interface/PositionJointInterface</hardwareInterface>
+      <mechanicalReduction>1</mechanicalReduction>
+    </actuator>
+  </transmission>
+  <transmission name="joint7_trans">
+    <type>transmission_interface/SimpleTransmission</type>
+    <joint name="joint7">
+      <hardwareInterface>hardware_interface/PositionJointInterface</hardwareInterface>
+    </joint>
+    <actuator name="joint7_motor">
+      <hardwareInterface>hardware_interface/PositionJointInterface</hardwareInterface>
+      <mechanicalReduction>1</mechanicalReduction>
+    </actuator>
+  </transmission>
 </robot>

Commit message: Enhance launch configuration for mobile manipulator; add RViz argument, improve URDF dimensions, and adjust material properties for better visualization in Gazebo.

File: MOBILE_MANIPULATOR/mobile_manipulator_description/urdf/linear_guide.xacro (robot description, xacro)
@@ -4,16 +4,16 @@
     <visual>
       <geometry>
-        <box size="0.1 0.1 1.0"/>
+        <box size="0.08 0.08 0.8"/>
       </geometry>
-      <origin xyz="0 -0.1 0.5" rpy="0 0 0"/>
+      <origin xyz="0 -0.1 0.37" rpy="0 0 0"/>
       <material name="grey">
-        <color rgba="0.5 0.5 0.5 1.0"/>
+        <color rgba="0.5 0.5 0.5 0.8"/>
       </material>
     </visual>
     <collision>
       <geometry>
-        <box size="0.1 0.1 1.0"/>
+        <box size="0.08 0.08 0.8"/>
       </geometry>
-      <origin xyz="0 -0.1 0.5" rpy="0 0 0"/>
+      <origin xyz="0 -0.1 0.37" rpy="0 0 0"/>
     </collision>
     <inertial>
@@ -22,4 +22,7 @@
     </inertial>
   </link>
+    <gazebo reference="column">
+      <material>Gazebo/Orange</material>
+  </gazebo>
   <link name="slider">
     <visual>
@@ -43,4 +46,7 @@
     </inertial>
   </link>
+ <gazebo reference="slider">
+      <material>Gazebo/Grey</material>
+  </gazebo>
   <joint name="slider_joint" type="prismatic">
     <parent link="column"/>
