Commit message: Added camera

File: MOBILE_MANIPULATOR/mobile_manipulator_description/urdf/camera_module.urdf.xacro (robot description, xacro)
@@ -6,5 +6,5 @@
     <link name="camera_link">
       <visual>
-        <origin xyz="0 0 0" rpy="0 0 0"/>
+        <origin xyz="0 0 0" rpy="1.57 0 1.57"/>
         <geometry>
           <!-- <box size="0.3 0.3 0.05"/>  -->

File: MOBILE_MANIPULATOR/mobile_manipulator_description/urdf/mobile_manipulator.urdf.xacro (robot description, xacro)
@@ -37,10 +37,10 @@
         </plugin>
     </gazebo>
-  <!-- <xacro:include filename="$(find mobile_manipulator_description)/urdf/camera_module.urdf.xacro"/>
+  <xacro:include filename="$(find mobile_manipulator_description)/urdf/camera_module.urdf.xacro"/>
   <xacro:intel_d435_camera/>
-  <joint name="link_7to_camera" type="fixed">
-    <parent link="Link7"/>
+  <joint name="sliderto_camera" type="fixed">
+    <parent link="slider"/>
     <child  link="camera_link"/>
-    <origin xyz="0.0 -0.05 0.0" rpy="0 0 0"/>
-  </joint> -->
+    <origin xyz="0 -0.5 0.1" rpy="0 0 -1.57"/>
+  </joint>
 </robot>
