Commit message: Added vision

File: MOBILE_MANIPULATOR/mobile_manipulator_description/urdf/mobile_manipulator.urdf.xacro (robot description, xacro)
@@ -22,3 +22,10 @@
     </plugin>
   </gazebo>
+  <!-- <xacro:include filename="$(find mobile_manipulator_description)/urdf/camera_module.urdf.xacro"/>
+  <xacro:intel_d435_camera/>
+  <joint name="link_7to_camera" type="fixed">
+    <parent link="Link7"/>
+    <child  link="camera_link"/>
+    <origin xyz="0.0 -0.05 0.0" rpy="0 0 0"/>
+  </joint> -->
 </robot>

Commit message: Added lif detector plugin

File: MOBILE_MANIPULATOR/mobile_manipulator_description/urdf/mobile_manipulator.urdf.xacro (robot description, xacro)
@@ -13,5 +13,5 @@
     <parent link="slider"/>
     <child  link="base_link"/>
-    <origin xyz="0 -0.33 0.06" rpy="0 0 0"/>
+    <origin xyz="0 -0.33 0.06" rpy="0 0 -1.57"/>
   </joint>
   <gazebo>
@@ -22,4 +22,22 @@
     </plugin>
   </gazebo>
+      <gazebo>
+        <plugin name="elevator_trigger_plugin" filename="libelevator_trigger_plugin.so">
+        <!-- Elevator entry position -->
+        <target_pose_enter>
+            <x>2.0</x>
+            <y>1.5</y>
+            <z>0.0</z>
+        </target_pose_enter>
+        <!-- Elevator exit position -->
+        <target_pose_exit>
+            <x>5.0</x>
+            <y>1.5</y>
+            <z>0.0</z>
+        </target_pose_exit>
+        <!-- Distance tolerance in meters -->
+        <tolerance>0.5</tolerance>
+        </plugin>
+    </gazebo>
   <!-- <xacro:include filename="$(find mobile_manipulator_description)/urdf/camera_module.urdf.xacro"/>
   <xacro:intel_d435_camera/>

Commit message: Update waypoint timings and adjust arm trajectory for smoother operation

File: MOBILE_MANIPULATOR/mobile_manipulator_description/urdf/mobile_manipulator.urdf.xacro (robot description, xacro)
@@ -13,5 +13,5 @@
     <parent link="slider"/>
     <child  link="base_link"/>
-    <origin xyz="0 -0.37 0.06" rpy="0 0 0"/>
+    <origin xyz="0 -0.33 0.06" rpy="0 0 0"/>
   </joint>
   <gazebo>
@@ -69,5 +69,5 @@
     <parent link="link_base"/>
     <child  link="camera_link_base"/>
-    <origin xyz="-0.3 -0.3 0.85" rpy="0 0 0"/>
+    <origin xyz="-0.3 0.3 0.85" rpy="0 0 0"/>
   </joint>
 </robot>
