Commit message: Refactored urdf of alphabot

File: ALPHA_BOT/alphabot_description/urdf/alphabot.urdf.xacro (robot description, xacro)
@@ -1,22 +1,13 @@
 <?xml version="1.0"?>
 <robot name="ackermann_logistic_robot" xmlns:xacro="http://www.ros.org/wiki/xacro">
-  <!-- Absolute path to the package share -->
-  <xacro:property name="alphabot_share" value="$(find alphabot_description)"/>
-  <!-- ============ base ============ -->
-  <!-- Move inertial off the root (removes KDL warning) -->
+  <!-- Where meshes are (URIs from SDF "model://" mapped to package path) -->
+  <xacro:property name="mesh_dir" value="$(find alphabot_description)/meshes"/>
+  <!-- ========== Base & Chassis (as in SDF) ========== -->
   <link name="base_link"/>
-  <link name="base_inertia_link">
-    <inertial>
-      <origin xyz="0 0 0" rpy="0 0 0"/>
-      <mass value="1.0"/>
-      <inertia ixx="0.1" ixy="0" ixz="0" iyy="0.1" iyz="0" izz="0.1"/>
-    </inertial>
-  </link>
-  <joint name="base_inertia_fixed" type="fixed">
+  <joint name="chassis_link_joint" type="fixed">
     <origin xyz="0 0 0" rpy="0 0 0"/>
     <parent link="base_link"/>
-    <child  link="base_inertia_link"/>
-  </joint>
-  <!-- Chassis fixed to base_link -->
+    <child  link="chassis_link"/>
+  </joint>
   <link name="chassis_link">
     <inertial>
@@ -25,66 +16,79 @@
       <inertia ixx="1997.86" ixy="-3e-05" ixz="-1e-06" iyy="442.769" iyz="62.5206" izz="2238.05"/>
     </inertial>
-    <visual>
-      <origin xyz="0 0 0" rpy="0 0 0"/>
-      <geometry>
-        <mesh filename="${alphabot_share}/meshes/chassis.dae" scale="0.5 0.5 0.5"/>
-      </geometry>
-    </visual>
-    <collision>
-      <origin xyz="0 0 0" rpy="0 0 0"/>
-      <geometry>
-        <mesh filename="${alphabot_share}/meshes/chassis.dae" scale="0.5 0.5 0.5"/>
-      </geometry>
-    </collision>
-  </link>
-  <joint name="chassis_link_joint" type="fixed">
-    <origin xyz="0 0 0" rpy="0 0 0"/>
-    <parent link="base_link"/>
-    <child link="chassis_link"/>
-  </joint>
-  <!-- ============ rear wheels (revolute about X) ============ -->
-  <link name="bl_1">
-    <inertial>
-      <origin xyz="0 0 0" rpy="0 0 0"/>
-      <mass value="24.5"/>
-      <inertia ixx="1.84514" ixy="0" ixz="0" iyy="1.04961" iyz="0" izz="1.04961"/>
-    </inertial>
-    <visual>
-      <origin xyz="0 0 0" rpy="0 1.5708 0"/>
-      <geometry><mesh filename="${alphabot_share}/meshes/wheel.dae" scale="0.5 0.5 0.5"/></geometry>
-    </visual>
-    <collision>
-      <origin xyz="0 0 0" rpy="0 1.5708 0"/>
-      <geometry><mesh filename="${alphabot_share}/meshes/wheel.dae" scale="0.5 0.5 0.5"/></geometry>
-    </collision>
-  </link>
+    <!-- visual == mesh (scale 0.5) -->
+    <visual name="chassis_link_visual">
+      <origin xyz="0 0 0.0" rpy="0 0 0"/>
+      <geometry>
+        <mesh filename="${mesh_dir}/chassis.dae" scale="0.5 0.5 0.5"/>
+      </geometry>
+    </visual>
+    <!-- collision == mesh (scale 0.5), like SDF -->
+    <collision name="chassis_link_collision">
+      <origin xyz="0 0 0.0" rpy="0 0 0"/>
+      <geometry>
+        <mesh filename="${mesh_dir}/chassis.dae" scale="0.5 0.5 0.5"/>
+      </geometry>
+    </collision>
+  </link>
+  <!-- ========== Rear Wheels (revolute in SDF; URDF: continuous, no limits) ========== -->
   <joint name="bl_axle" type="continuous">
     <origin xyz="-0.18 -0.244 0.0" rpy="0 0 0"/>
     <parent link="chassis_link"/>
-    <child link="bl_1"/>
-    <axis xyz="1 0 0"/>
-  </joint>
-  <link name="br_1">
-    <inertial>
-      <origin xyz="-0.0377 0 0" rpy="0 0 0"/>
-      <mass value="24.5"/>
-      <inertia ixx="1.84514" ixy="0" ixz="0" iyy="1.04961" iyz="0" izz="1.04961"/>
-    </inertial>
-    <visual>
-      <origin xyz="0 0 0" rpy="0 1.5708 0"/>
-      <geometry><mesh filename="${alphabot_share}/meshes/wheel.dae" scale="0.5 0.5 0.5"/></geometry>
-    </visual>
-    <collision>
-      <origin xyz="0 0 0" rpy="0 1.5708 0"/>
-      <geometry><mesh filename="${alphabot_share}/meshes/wheel.dae" scale="0.5 0.5 0.5"/></geometry>
-    </collision>
+    <child  link="bl_1"/>
+    <axis xyz="-1 0 0"/>
+    <dynamics friction="12.031606150200002"/>
+  </joint>
+  <link name="bl_1">
+    <inertial>
+      <origin xyz="0 0 0" rpy="0 0 0"/>
+      <mass value="24.5"/>
+      <inertia ixx="1.84514" ixy="0" ixz="0" iyy="1.04961" iyz="0" izz="1.04961"/>
+    </inertial>
+    <!-- collision == cylinder (pose same as SDF collision) -->
+    <collision name="bl_1_collision">
+      <origin xyz="0 0 0" rpy="0 1.5708 0"/>
+      <geometry><cylinder radius="0.072" length="0.06"/></geometry>
+    </collision>
+    <!-- visual == mesh wheel (scale 0.5), so it shows up -->
+    <visual name="bl_1_visual">
+      <origin xyz="0 0 0" rpy="0 0 0"/>
+      <geometry>
+        <mesh filename="${mesh_dir}/wheel.dae" scale="0.5 0.5 0.5"/>
+      </geometry>
+    </visual>
   </link>
   <joint name="br_axle" type="continuous">
     <origin xyz="0.18 -0.244 0.0" rpy="0 0 0"/>
     <parent link="chassis_link"/>
-    <child link="br_1"/>
-    <axis xyz="1 0 0"/>
-  </joint>
-  <!-- ============ steering knuckles (revolute about Z) ============ -->
+    <child  link="br_1"/>
+    <axis xyz="-1 0 0"/>
+    <dynamics friction="12.031606150200002"/>
+  </joint>
+  <link name="br_1">
+    <inertial>
+      <origin xyz="-0.0377 0 0" rpy="0 0 0"/>
+      <mass value="24.5"/>
+      <inertia ixx="1.84514" ixy="0" ixz="0" iyy="1.04961" iyz="0" izz="1.04961"/>
+    </inertial>
+    <collision name="br_1_collision">
+      <origin xyz="0 0 0" rpy="0 1.5708 0"/>
+      <geometry><cylinder radius="0.072" length="0.06"/></geometry>
+    </collision>
+    <visual name="br_1_visual">
+      <origin xyz="0 0 0" rpy="0 0 0"/>
+      <geometry>
+        <mesh filename="${mesh_dir}/wheel.dae" scale="0.5 0.5 0.5"/>
+      </geometry>
+    </visual>
+  </link>
+  <!-- ========== Steering Knuckles (revolute with limits, as SDF) ========== -->
+  <joint name="l_steer" type="revolute">
+    <origin xyz="-0.236 0.244 0.0" rpy="0 0 0"/>
+    <parent link="chassis_link"/>
+    <child  link="l_steer_1"/>
+    <axis xyz="0 0 1"/>
+    <limit lower="-0.95" upper="0.95" effort="1e9" velocity="1e9"/>
+    <dynamics friction="18.0474092253"/>
+  </joint>
   <link name="l_steer_1">
     <inertial>
@@ -94,10 +98,11 @@
     </inertial>
   </link>
-  <joint name="l_steer" type="revolute">
-    <origin xyz="-0.236 0.244 0.0" rpy="0 0 0"/>
-    <parent link="chassis_link"/>
-    <child link="l_steer_1"/>
+  <joint name="r_steer" type="revolute">
+    <origin xyz="0.236 0.244 0.0" rpy="0 0 0"/>
+    <parent link="chassis_link"/>
+    <child  link="r_steer_1"/>
     <axis xyz="0 0 1"/>
-    <limit lower="-0.95" upper="0.95" effort="100.0" velocity="5.0"/>
+    <limit lower="-0.95" upper="0.95" effort="1e9" velocity="1e9"/>
+    <dynamics damping="0.01" friction="18.0474092253"/>
   </joint>
   <link name="r_steer_1">
@@ -108,38 +113,13 @@
     </inertial>
   </link>
-  <joint name="r_steer" type="revolute">
-    <origin xyz="0.236 0.244 0.0" rpy="0 0 0"/>
-    <parent link="chassis_link"/>
-    <child link="r_steer_1"/>
-    <axis xyz="0 0 1"/>
-    <limit lower="-0.95" upper="0.95" effort="100.0" velocity="5.0"/>
-  </joint>
-  <!-- ============ front wheels (rotate about X) ============ -->
-  <link name="fl_1">
-    <inertial>
-      <origin xyz="-0.0377 0 0" rpy="0 0 0"/>
-      <mass value="24.5"/>
-      <inertia ixx="1.84514" ixy="0" ixz="0" iyy="1.04961" iyz="0" izz="1.04961"/>
-    </inertial>
-    <visual>
-      <origin xyz="0 0 0" rpy="0 1.5708 0"/>
-      <geometry>
-      <mesh filename="${alphabot_share}/meshes/wheel.dae" scale="0.5 0.5 0.5"/>
-      </geometry>
-    </visual>
-    <collision>
-      <origin xyz="0 0 0" rpy="0 1.5708 0"/>
-      <geometry>
-      <mesh filename="${alphabot_share}/meshes/wheel.dae" scale="0.5 0.5 0.5"/>
-      </geometry>
-    </collision>
-  </link>
+  <!-- ========== Front Wheels (continuous) ========== -->
   <joint name="fl_axle" type="continuous">
     <origin xyz="0 0 0" rpy="0 0 0"/>
     <parent link="l_steer_1"/>
-    <child link="fl_1"/>
-    <axis xyz="1 0 0"/>
-  </joint>
-  <link name="fr_1">
+    <child  link="fl_1"/>
+    <axis xyz="-1 0 0"/>
+    <dynamics friction="12.031606150200002"/>
+  </joint>
+  <link name="fl_1">
     <inertial>
       <origin xyz="-0.0377 0 0" rpy="0 0 0"/>
@@ -147,24 +127,40 @@
       <inertia ixx="1.84514" ixy="0" ixz="0" iyy="1.04961" iyz="0" izz="1.04961"/>
     </inertial>
-    <visual>
-      <origin xyz="0 0 0" rpy="0 1.5708 0"/>
-      <geometry>
-      <mesh filename="${alphabot_share}/meshes/wheel.dae" scale="0.5 0.5 0.5"/>
-      </geometry>
-    </visual>
-    <collision>
-      <origin xyz="0 0 0" rpy="0 1.5708 0"/>
-      <geometry>
-      <mesh filename="${alphabot_share}/meshes/wheel.dae" scale="0.5 0.5 0.5"/>
-      </geometry>
-    </collision>
+    <collision name="fl_1_collision">
+      <origin xyz="0 0 0" rpy="0 1.5708 0"/>
+      <geometry><cylinder radius="0.072" length="0.06"/></geometry>
+    </collision>
+    <visual name="fl_1_visual">
+      <origin xyz="0 0 0" rpy="0 0 0"/>
+      <geometry>
+        <mesh filename="${mesh_dir}/wheel.dae" scale="0.5 0.5 0.5"/>
+      </geometry>
+    </visual>
   </link>
   <joint name="fr_axle" type="continuous">
     <origin xyz="0 0 0" rpy="0 0 0"/>
     <parent link="r_steer_1"/>
-    <child link="fr_1"/>
-    <axis xyz="1 0 0"/>
-  </joint>
-  <!-- ============ platform / lift (fixed) ============ -->
+    <child  link="fr_1"/>
+    <axis xyz="-1 0 0"/>
+    <dynamics friction="12.031606150200002"/>
+  </joint>
+  <link name="fr_1">
+    <inertial>
+      <origin xyz="-0.0377 0 0" rpy="0 0 0"/>
+      <mass value="24.5"/>
+      <inertia ixx="1.84514" ixy="0" ixz="0" iyy="1.04961" iyz="0" izz="1.04961"/>
+    </inertial>
+    <collision name="fr_1_collision">
+      <origin xyz="0 0 0" rpy="0 1.5708 0"/>
+      <geometry><cylinder radius="0.072" length="0.06"/></geometry>
+    </collision>
+    <visual name="fr_1_visual">
+      <origin xyz="0 0 0" rpy="0 0 0"/>
+      <geometry>
+        <mesh filename="${mesh_dir}/wheel.dae" scale="0.5 0.5 0.5"/>
+      </geometry>
+    </visual>
+  </link>
+  <!-- ========== Lift (prismatic, limits as SDF) ========== -->
   <link name="lift_link">
     <inertial>
@@ -176,5 +172,5 @@
       <origin xyz="0 0 0.1" rpy="0 0 0"/>
       <geometry>
-        <mesh filename="${alphabot_share}/meshes/platform.dae" scale="0.5 0.5 0.5"/>
+        <mesh filename="${mesh_dir}/platform.dae" scale="0.5 0.5 0.5"/>
       </geometry>
     </visual>
@@ -191,39 +187,31 @@
     <child link="lift_link"/>
   </joint>
-  <!-- ============ Gazebo (Classic) tags ============ -->
-  <gazebo reference="fl_1">
-    <visual>
-      <geometry>
-        <mesh filename="${alphabot_share}/meshes/wheel.dae" scale="0.5 0.5 0.5"/>
-      </geometry>
-    </visual>
+  <!-- ========== Gazebo Classic extensions (from your SDF surfaces) ========== -->
+  <!-- Chassis friction + self-collide -->
+  <gazebo reference="chassis_link">
+    <selfCollide>true</selfCollide>
+    <mu1>0.2</mu1>
+    <mu2>0.2</mu2>
   </gazebo>
-  <gazebo reference="fr_1">
-    <visual>
-      <geometry>
-        <mesh filename="${alphabot_share}/meshes/wheel.dae" scale="0.5 0.5 0.5"/>
-      </geometry>
-    </visual>
+  <!-- Wheel high friction -->
+  <gazebo reference="bl_1"><mu1>1000000</mu1><mu2>1000000</mu2></gazebo>
+  <gazebo reference="br_1"><mu1>1000000</mu1><mu2>1000000</mu2></gazebo>
+  <gazebo reference="fl_1"><mu1>1000000</mu1><mu2>1000000</mu2></gazebo>
+  <gazebo reference="fr_1"><mu1>1000000</mu1><mu2>1000000</mu2></gazebo>
+  <!-- Lift contact/friction intents -->
+  <gazebo reference="lift_link">
+    <mu1>1000000</mu1>
+    <mu2>100000</mu2>
+    <kp>1e5</kp>
+    <kd>1</kd>
+    <maxVel>0.01</maxVel>
+    <minDepth>0.001</minDepth>
   </gazebo>
-  <gazebo reference="bl_1">
-    <visual>
-      <geometry>
-        <mesh filename="${alphabot_share}/meshes/wheel.dae" scale="0.5 0.5 0.5"/>
-      </geometry>
-    </visual>
-  </gazebo>
-  <gazebo reference="br_1">
-    <visual>
-      <geometry>
-        <mesh filename="${alphabot_share}/meshes/wheel.dae" scale="0.5 0.5 0.5"/>
-      </geometry>
-    </visual>
-  </gazebo>
-  <!-- Ackermann drive plugin -->
+  <!-- ========== Ackermann Drive Plugin (exactly as in your SDF) ========== -->
   <gazebo>
     <plugin name="ackermann_drive" filename="libgazebo_ros_ackermann_drive.so">
       <ros>
-        <remapping>cmd_vel:=cmd_vel</remapping>
-        <remapping>odom:=odom</remapping>
+        <remapping>cmd_vel:=/amazon_robot/cmd_vel</remapping>
+        <remapping>odom:=/amazon_robot/odom</remapping>
         <remapping>distance:=distance</remapping>
       </ros>
@@ -237,5 +225,5 @@
       <max_steer>0.52</max_steer>
       <max_steering_angle>0.64</max_steering_angle>
-      <max_speed>50.0</max_speed>
+      <max_speed>50</max_speed>
       <left_steering_pid_gain>1500 900 450</left_steering_pid_gain>
       <left_steering_i_range>0 0</left_steering_i_range>
