Commit message: Backup

File: ALPHA_BOT/alphabot_description/urdf/alphabot.urdf.xacro (robot description, xacro)
@@ -7,39 +7,69 @@
   <xacro:property name="odom_topic"        value="/amazon_robot/odom"/>
   <xacro:property name="scan_topic"        value="/scan"/>
-  <!-- ================== Base & Chassis ================== -->
+  <!-- ================== Frames (TF root) ================== -->
+  <link name="base_footprint"/>
   <link name="base_link"/>
+  <joint name="base_joint" type="fixed">
+    <parent link="base_footprint"/>
+    <child  link="base_link"/>
+    <!-- raise base_link so footprint sits at ground; wheel_radius=0.072 -->
+    <origin xyz="0 0 0.072" rpy="0 0 0"/>
+  </joint>
+  <!-- ================== Chassis ================== -->
+  <link name="chassis_link">
+    <inertial>
+      <origin xyz="0 0 0" rpy="0 0 0"/>
+      <mass value="1580"/>
+      <!-- (placeholder inertia) -->
+      <inertia ixx="1997.86" ixy="0" ixz="0" iyy="442.769" iyz="62.5206" izz="2238.05"/>
+    </inertial>
+    <visual>
+      <origin xyz="0 0 0" rpy="0 0 0"/>
+      <geometry>
+        <mesh filename="${pkg_share}/meshes/chassis.dae" scale="0.5 0.5 0.5"/>
+      </geometry>
+    </visual>
+    <collision>
+      <origin xyz="0 0 0" rpy="0 0 0"/>
+      <geometry>
+        <mesh filename="${pkg_share}/meshes/chassis.dae" scale="0.5 0.5 0.5"/>
+      </geometry>
+    </collision>
+  </link>
   <joint name="chassis_link_joint" type="fixed">
-    <origin xyz="0 0 0" rpy="0 0 0"/>
     <parent link="base_link"/>
     <child  link="chassis_link"/>
-  </joint>
-  <link name="chassis_link">
-    <inertial>
-      <origin xyz="1e-06 0.07307 0.65096" rpy="0 0 0"/>
-      <mass value="1580"/>
-      <inertia ixx="1997.86" ixy="-3e-05" ixz="-1e-06" iyy="442.769" iyz="62.5206" izz="2238.05"/>
-    </inertial>
-    <visual name="chassis_link_visual">
-      <origin xyz="0 0 0.0" rpy="0 0 0"/>
-      <geometry>
-        <mesh filename="${pkg_share}/meshes/chassis.dae" scale="0.5 0.5 0.5"/>
-      </geometry>
-    </visual>
-    <collision name="chassis_link_collision">
-      <origin xyz="0 0 0.0" rpy="0 0 0"/>
-      <geometry>
-        <mesh filename="${pkg_share}/meshes/chassis.dae" scale="0.5 0.5 0.5"/>
-      </geometry>
-    </collision>
-  </link>
-  <!-- ================== Rear Wheels ================== -->
+    <origin xyz="0 0 0" rpy="0 0 0"/>
+  </joint>
+  <!-- ================== Wheels ================== -->
+  <!-- Shared wheel params: radius=0.072, width=0.06; we orient cyl axis along X (rpy 0 1.5708 0) -->
+  <!-- Rear LEFT (drive) -->
+  <link name="bl_1">
+    <inertial>
+      <origin xyz="0 0 0" rpy="0 0 0"/>
+      <mass value="24.5"/>
+      <inertia ixx="1.84514" ixy="0" ixz="0" iyy="1.04961" iyz="0" izz="1.04961"/>
+    </inertial>
+    <collision>
+      <origin xyz="0 0 0" rpy="0 1.5708 0"/>
+      <geometry><cylinder radius="0.072" length="0.06"/></geometry>
+    </collision>
+    <visual>
+      <origin xyz="0 0 0" rpy="0 0 0"/>
+      <geometry>
+        <mesh filename="${pkg_share}/meshes/wheel.dae" scale="0.5 0.5 0.5"/>
+      </geometry>
+    </visual>
+  </link>
   <joint name="bl_axle" type="continuous">
-    <origin xyz="-0.18 -0.244 0.0" rpy="0 0 0"/>
+    <origin xyz="-0.18 -0.244 0" rpy="0 0 0"/>
     <parent link="chassis_link"/>
     <child  link="bl_1"/>
-    <axis xyz="-1 0 0"/>
-    <dynamics friction="12.031606150200002"/>
-  </joint>
-  <link name="bl_1">
+    <!-- rotate around X (matches collision orientation) -->
+    <axis xyz="1 0 0"/>
+    <dynamics friction="12.0316061502"/>
+  </joint>
+  <!-- Rear RIGHT (drive) -->
+  <link name="br_1">
     <inertial>
       <origin xyz="0 0 0" rpy="0 0 0"/>
@@ -47,9 +77,9 @@
       <inertia ixx="1.84514" ixy="0" ixz="0" iyy="1.04961" iyz="0" izz="1.04961"/>
     </inertial>
-    <collision name="bl_1_collision">
+    <collision>
       <origin xyz="0 0 0" rpy="0 1.5708 0"/>
       <geometry><cylinder radius="0.072" length="0.06"/></geometry>
     </collision>
-    <visual name="bl_1_visual">
+    <visual>
       <origin xyz="0 0 0" rpy="0 0 0"/>
       <geometry>
@@ -59,30 +89,16 @@
   </link>
   <joint name="br_axle" type="continuous">
-    <origin xyz="0.18 -0.244 0.0" rpy="0 0 0"/>
+    <origin xyz="0.18 -0.244 0" rpy="0 0 0"/>
     <parent link="chassis_link"/>
     <child  link="br_1"/>
-    <axis xyz="-1 0 0"/>
-    <dynamics friction="12.031606150200002"/>
-  </joint>
-  <link name="br_1">
-    <inertial>
-      <origin xyz="-0.0377 0 0" rpy="0 0 0"/>
-      <mass value="24.5"/>
-      <inertia ixx="1.84514" ixy="0" ixz="0" iyy="1.04961" iyz="0" izz="1.04961"/>
-    </inertial>
-    <collision name="br_1_collision">
-      <origin xyz="0 0 0" rpy="0 1.5708 0"/>
-      <geometry><cylinder radius="0.072" length="0.06"/></geometry>
-    </collision>
-    <visual name="br_1_visual">
-      <origin xyz="0 0 0" rpy="0 0 0"/>
-      <geometry>
-        <mesh filename="${pkg_share}/meshes/wheel.dae" scale="0.5 0.5 0.5"/>
-      </geometry>
-    </visual>
-  </link>
-  <!-- ================== Front (steering locked) ================== -->
+    <axis xyz="1 0 0"/>
+    <dynamics friction="12.0316061502"/>
+  </joint>
+  <!-- Front locked “steer” carriers (fixed at 0 rad) -->
+  <link name="l_steer_1">
+    <inertial><origin xyz="0 0 0"/><mass value="1"/><inertia ixx="1" ixy="0" ixz="0" iyy="1" iyz="0" izz="1"/></inertial>
+  </link>
   <joint name="l_steer" type="revolute">
-    <origin xyz="-0.236 0.244 0.0" rpy="0 0 0"/>
+    <origin xyz="-0.236 0.244 0" rpy="0 0 0"/>
     <parent link="chassis_link"/>
     <child  link="l_steer_1"/>
@@ -90,13 +106,9 @@
     <limit lower="0.0" upper="0.0" effort="1e9" velocity="0.0"/>
   </joint>
-  <link name="l_steer_1">
-    <inertial>
-      <origin xyz="0.003381 0 0.02162" rpy="0 0 0"/>
-      <mass value="1"/>
-      <inertia ixx="1" ixy="0" ixz="0" iyy="1" iyz="0" izz="1"/>
-    </inertial>
+  <link name="r_steer_1">
+    <inertial><origin xyz="0 0 0"/><mass value="1"/><inertia ixx="1" ixy="0" ixz="0" iyy="1" iyz="0" izz="1"/></inertial>
   </link>
   <joint name="r_steer" type="revolute">
-    <origin xyz="0.236 0.244 0.0" rpy="0 0 0"/>
+    <origin xyz="0.236 0.244 0" rpy="0 0 0"/>
     <parent link="chassis_link"/>
     <child  link="r_steer_1"/>
@@ -104,10 +116,21 @@
     <limit lower="0.0" upper="0.0" effort="1e9" velocity="0.0"/>
   </joint>
-  <link name="r_steer_1">
-    <inertial>
-      <origin xyz="0.003381 0 0.02162" rpy="0 0 0"/>
-      <mass value="1"/>
-      <inertia ixx="1" ixy="0" ixz="0" iyy="1" iyz="0" izz="1"/>
-    </inertial>
+  <!-- Front LEFT (idler) -->
+  <link name="fl_1">
+    <inertial>
+      <origin xyz="0 0 0" rpy="0 0 0"/>
+      <mass value="24.5"/>
+      <inertia ixx="1.84514" ixy="0" ixz="0" iyy="1.04961" iyz="0" izz="1.04961"/>
+    </inertial>
+    <collision>
+      <origin xyz="0 0 0" rpy="0 1.5708 0"/>
+      <geometry><cylinder radius="0.072" length="0.06"/></geometry>
+    </collision>
+    <visual>
+      <origin xyz="0 0 0" rpy="0 0 0"/>
+      <geometry>
+        <mesh filename="${pkg_share}/meshes/wheel.dae" scale="0.5 0.5 0.5"/>
+      </geometry>
+    </visual>
   </link>
   <joint name="fl_axle" type="continuous">
@@ -115,17 +138,18 @@
     <parent link="l_steer_1"/>
     <child  link="fl_1"/>
-    <axis xyz="-1 0 0"/>
-  </joint>
-  <link name="fl_1">
-    <inertial>
-      <origin xyz="-0.0377 0 0" rpy="0 0 0"/>
+    <axis xyz="1 0 0"/>
+  </joint>
+  <!-- Front RIGHT (idler) -->
+  <link name="fr_1">
+    <inertial>
+      <origin xyz="0 0 0" rpy="0 0 0"/>
       <mass value="24.5"/>
       <inertia ixx="1.84514" ixy="0" ixz="0" iyy="1.04961" iyz="0" izz="1.04961"/>
     </inertial>
-    <collision name="fl_1_collision">
+    <collision>
       <origin xyz="0 0 0" rpy="0 1.5708 0"/>
       <geometry><cylinder radius="0.072" length="0.06"/></geometry>
     </collision>
-    <visual name="fl_1_visual">
+    <visual>
       <origin xyz="0 0 0" rpy="0 0 0"/>
       <geometry>
@@ -138,23 +162,6 @@
     <parent link="r_steer_1"/>
     <child  link="fr_1"/>
-    <axis xyz="-1 0 0"/>
-  </joint>
-  <link name="fr_1">
-    <inertial>
-      <origin xyz="-0.0377 0 0" rpy="0 0 0"/>
-      <mass value="24.5"/>
-      <inertia ixx="1.84514" ixy="0" ixz="0" iyy="1.04961" iyz="0" izz="1.04961"/>
-    </inertial>
-    <collision name="fr_1_collision">
-      <origin xyz="0 0 0" rpy="0 1.5708 0"/>
-      <geometry><cylinder radius="0.072" length="0.06"/></geometry>
-    </collision>
-    <visual name="fr_1_visual">
-      <origin xyz="0 0 0" rpy="0 0 0"/>
-      <geometry>
-        <mesh filename="${pkg_share}/meshes/wheel.dae" scale="0.5 0.5 0.5"/>
-      </geometry>
-    </visual>
-  </link>
+    <axis xyz="1 0 0"/>
+  </joint>
   <!-- ================== LiDAR & Lift ================== -->
   <link name="lidar_link">
@@ -163,37 +170,85 @@
     <collision><origin xyz="0 0 0"/><geometry><cylinder radius="0.04" length="0.05"/></geometry></collision>
   </link>
-  <joint name="lidar_joint" type="fixed"><origin xyz="0 0 0.18"/><parent link="base_link"/><child link="lidar_link"/></joint>
+  <joint name="lidar_joint" type="fixed">
+    <origin xyz="0 0 0.18" rpy="0 0 0"/>
+    <parent link="base_link"/>
+    <child  link="lidar_link"/>
+  </joint>
   <link name="lift_link">
     <inertial><origin xyz="0 0 0"/><mass value="0.1"/><inertia ixx="0.001" ixy="0" ixz="0" iyy="0.001" iyz="0" izz="0.001"/></inertial>
     <visual>
-      <origin xyz="0 0 0.1"/>
-      <geometry><mesh filename="${pkg_share}/meshes/platform.dae" scale="0.5 0.5 0.5"/></geometry>
-    </visual>
-    <collision><origin xyz="0 0 0"/><geometry><box size="0.2805 0.2 0.03"/></geometry></collision>
-  </link>
-  <joint name="lift_fixed_joint" type="fixed"><origin xyz="0 0 0.02"/><parent link="lidar_link"/><child link="lift_link"/></joint>
+      <origin xyz="0 0 0.1" rpy="0 0 0"/>
+      <geometry>
+        <mesh filename="${pkg_share}/meshes/platform.dae" scale="0.5 0.5 0.5"/>
+      </geometry>
+    </visual>
+    <collision>
+      <origin xyz="0 0 0" rpy="0 0 0"/>
+      <geometry><box size="0.2805 0.2 0.03"/></geometry>
+    </collision>
+  </link>
+  <joint name="lift_fixed_joint" type="fixed">
+    <origin xyz="0 0 0.02" rpy="0 0 0"/>
+    <parent link="lidar_link"/>
+    <child  link="lift_link"/>
+  </joint>
   <!-- ================== Camera frames ================== -->
-  <link name="camera_mount_link"><inertial><origin xyz="0 0 0"/><mass value="0.1"/><inertia ixx="1e-4" ixy="0" ixz="0" iyy="1e-4" iyz="0" izz="1e-4"/></inertial></link>
-  <joint name="camera_mount_joint" type="fixed"><origin xyz="0 0.45 0.09"/><parent link="base_link"/><child link="camera_mount_link"/></joint>
-  <link name="camera_link"/><joint name="camera_joint" type="fixed"><parent link="camera_mount_link"/><child link="camera_link"/></joint>
-  <link name="camera_optical_frame"/><joint name="camera_optical_joint" type="fixed"><origin rpy="0 -1.57079632679 3.14159265359"/><parent link="camera_link"/><child link="camera_optical_frame"/></joint>
-  <!-- ================== Gazebo Classic bits ================== -->
+  <link name="camera_mount_link">
+    <inertial><origin xyz="0 0 0"/><mass value="0.1"/><inertia ixx="0.0001" ixy="0" ixz="0" iyy="0.0001" iyz="0" izz="0.0001"/></inertial>
+  </link>
+  <joint name="camera_mount_joint" type="fixed">
+    <origin xyz="0 0.45 0.09" rpy="0 0 0"/>
+    <parent link="base_link"/>
+    <child  link="camera_mount_link"/>
+  </joint>
+  <link name="camera_link"/>
+  <joint name="camera_joint" type="fixed">
+    <parent link="camera_mount_link"/>
+    <child  link="camera_link"/>
+    <origin xyz="0 0 0" rpy="0 0 0"/>
+  </joint>
+  <link name="camera_optical_frame"/>
+  <joint name="camera_optical_joint" type="fixed">
+    <origin xyz="0 0 0" rpy="0 -1.57079632679 3.14159265359"/>
+    <parent link="camera_link"/>
+    <child  link="camera_optical_frame"/>
+  </joint>
+  <!-- ================== Gazebo materials/contacts ================== -->
   <gazebo reference="chassis_link"><selfCollide>true</selfCollide><mu1>0.2</mu1><mu2>0.2</mu2></gazebo>
-  <gazebo reference="bl_1"><mu1>1000000</mu1><mu2>1000000</mu2></gazebo>
-  <gazebo reference="br_1"><mu1>1000000</mu1><mu2>1000000</mu2></gazebo>
-  <gazebo reference="fl_1"><mu1>1000000</mu1><mu2>1000000</mu2></gazebo>
-  <gazebo reference="fr_1"><mu1>1000000</mu1><mu2>1000000</mu2></gazebo>
-  <gazebo reference="lift_link"><mu1>1000000</mu1><mu2>100000</mu2><kp>1e5</kp><kd>1</kd><maxVel>0.01</maxVel><minDepth>0.001</minDepth></gazebo>
-  <!-- LiDAR sensor -->
+  <gazebo reference="bl_1"><mu1>1e6</mu1><mu2>1e6</mu2></gazebo>
+  <gazebo reference="br_1"><mu1>1e6</mu1><mu2>1e6</mu2></gazebo>
+  <gazebo reference="fl_1"><mu1>1e6</mu1><mu2>1e6</mu2></gazebo>
+  <gazebo reference="fr_1"><mu1>1e6</mu1><mu2>1e6</mu2></gazebo>
+  <gazebo reference="lift_link"><mu1>1e6</mu1><mu2>1e5</mu2><kp>1e5</kp><kd>1</kd><maxVel>0.01</maxVel><minDepth>0.001</minDepth></gazebo>
+  <!-- ================== Gazebo: LIDAR ================== -->
   <gazebo reference="lidar_link">
     <sensor name="lidar" type="ray">
-      <always_on>true</always_on><update_rate>20</update_rate><visualize>true</visualize>
+      <always_on>true</always_on>
+      <update_rate>20</update_rate>
+      <visualize>true</visualize>
       <ray>
-        <scan><horizontal><samples>720</samples><resolution>1</resolution><min_angle>-3.14159265</min_angle><max_angle>3.14159265</max_angle></horizontal></scan>
-        <range><min>0.12</min><max>30.0</max><resolution>0.01</resolution></range>
-        <noise><type>gaussian</type><mean>0.0</mean><stddev>0.01</stddev></noise>
+        <scan>
+          <horizontal>
+            <samples>720</samples>
+            <resolution>1</resolution>
+            <min_angle>-3.14159265</min_angle>
+            <max_angle>3.14159265</max_angle>
+          </horizontal>
+        </scan>
+        <range>
+          <min>0.12</min>
+          <max>30.0</max>
+          <resolution>0.01</resolution>
+        </range>
+        <noise>
+          <type>gaussian</type>
+          <mean>0.0</mean>
+          <stddev>0.01</stddev>
+        </noise>
       </ray>
       <plugin name="gazebo_ros_ray_sensor" filename="libgazebo_ros_ray_sensor.so">
-        <ros><remapping>~/out:=${scan_topic}</remapping></ros>
+        <ros>
+          <remapping>~/out:=$(arg scan_topic)</remapping>
+        </ros>
         <output_type>sensor_msgs/LaserScan</output_type>
         <frame_name>lidar_link</frame_name>
@@ -201,6 +256,6 @@
     </sensor>
   </gazebo>
-  <!-- Sim camera (optional) -->
-  <xacro:if value="${use_gazebo_camera}">
+  <!-- ================== Gazebo: camera (optional) ================== -->
+  <xacro:if value="$(arg use_gazebo_camera)">
     <gazebo reference="camera_link">
       <sensor name="sim_camera" type="camera">
@@ -208,5 +263,9 @@
         <camera>
           <horizontal_fov>1.39626</horizontal_fov>
-          <image><width>640</width><height>480</height><format>R8G8B8</format></image>
+          <image>
+            <width>640</width>
+            <height>480</height>
+            <format>R8G8B8</format>
+          </image>
           <clip><near>0.02</near><far>50.0</far></clip>
         </camera>
@@ -221,24 +280,26 @@
     </gazebo>
   </xacro:if>
-  <!-- Make sure joint states publish (helps TF) -->
+  <!-- ================== Gazebo: joint state publisher ================== -->
   <gazebo>
     <plugin name="joint_state_publisher" filename="libgazebo_ros_joint_state_publisher.so">
-      <ros/><update_rate>50</update_rate>
-      <joint_name>bl_axle</joint_name><joint_name>br_axle</joint_name>
-      <joint_name>fl_axle</joint_name><joint_name>fr_axle</joint_name>
-      <joint_name>l_steer</joint_name><joint_name>r_steer</joint_name>
+      <update_rate>50</update_rate>
+      <joint_name>bl_axle</joint_name>
+      <joint_name>br_axle</joint_name>
+      <joint_name>fl_axle</joint_name>
+      <joint_name>fr_axle</joint_name>
+      <joint_name>l_steer</joint_name>
+      <joint_name>r_steer</joint_name>
     </plugin>
   </gazebo>
-  <!-- Differential drive -->
+  <!-- ================== Gazebo: differential drive ================== -->
   <gazebo>
     <plugin name="diff_drive" filename="libgazebo_ros_diff_drive.so">
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
Commit message: Aded camera model

File: ALPHA_BOT/alphabot_description/urdf/alphabot.urdf.xacro (robot description, xacro)
@@ -1,11 +1,8 @@
 <?xml version="1.0"?>
 <robot name="alphabot" xmlns:xacro="http://www.ros.org/wiki/xacro">
-  <!-- Resolve the package share to an ABSOLUTE path -->
-  <xacro:property name="pkg_share" value="$(find alphabot_description)"/>
   <xacro:property name="use_gazebo_camera" value="true"/>
   <xacro:property name="cmd_vel_topic"     value="/amazon_robot/cmd_vel"/>
   <xacro:property name="odom_topic"        value="/amazon_robot/odom"/>
   <xacro:property name="scan_topic"        value="/scan"/>
-  <!-- ================== Frames (TF root) ================== -->
   <link name="base_footprint"/>
   <link name="base_link"/>
@@ -13,13 +10,10 @@
     <parent link="base_footprint"/>
     <child  link="base_link"/>
-    <!-- raise base_link so footprint sits at ground; wheel_radius=0.072 -->
     <origin xyz="0 0 0.072" rpy="0 0 0"/>
   </joint>
-  <!-- ================== Chassis ================== -->
   <link name="chassis_link">
     <inertial>
       <origin xyz="0 0 0" rpy="0 0 0"/>
       <mass value="1580"/>
-      <!-- (placeholder inertia) -->
       <inertia ixx="1997.86" ixy="0" ixz="0" iyy="442.769" iyz="62.5206" izz="2238.05"/>
     </inertial>
@@ -27,11 +21,11 @@
       <origin xyz="0 0 0" rpy="0 0 0"/>
       <geometry>
-        <mesh filename="${pkg_share}/meshes/chassis.dae" scale="0.5 0.5 0.5"/>
-      </geometry>
-    </visual>
-    <collision>
-      <origin xyz="0 0 0" rpy="0 0 0"/>
-      <geometry>
-        <mesh filename="${pkg_share}/meshes/chassis.dae" scale="0.5 0.5 0.5"/>
+        <mesh filename="package://alphabot_description/meshes/chassis.dae" scale="0.5 0.5 0.5"/>
+      </geometry>
+    </visual>
+    <collision>
+      <origin xyz="0 0 0" rpy="0 0 0"/>
+      <geometry>
+        <mesh filename="package://alphabot_description/meshes/chassis.dae" scale="0.5 0.5 0.5"/>
       </geometry>
     </collision>
@@ -58,5 +52,5 @@
       <origin xyz="0 0 0" rpy="0 0 0"/>
       <geometry>
-        <mesh filename="${pkg_share}/meshes/wheel.dae" scale="0.5 0.5 0.5"/>
+        <mesh filename="package://alphabot_description/meshes/wheel.dae" scale="0.5 0.5 0.5"/>
       </geometry>
     </visual>
@@ -66,9 +60,7 @@
     <parent link="chassis_link"/>
     <child  link="bl_1"/>
-    <!-- rotate around X (matches collision orientation) -->
     <axis xyz="1 0 0"/>
     <dynamics friction="12.0316061502"/>
   </joint>
-  <!-- Rear RIGHT (drive) -->
   <link name="br_1">
     <inertial>
@@ -84,5 +76,5 @@
       <origin xyz="0 0 0" rpy="0 0 0"/>
       <geometry>
-        <mesh filename="${pkg_share}/meshes/wheel.dae" scale="0.5 0.5 0.5"/>
+        <mesh filename="package://alphabot_description/meshes/wheel.dae" scale="0.5 0.5 0.5"/>
       </geometry>
     </visual>
@@ -95,5 +87,4 @@
     <dynamics friction="12.0316061502"/>
   </joint>
-  <!-- Front locked “steer” carriers (fixed at 0 rad) -->
   <link name="l_steer_1">
     <inertial><origin xyz="0 0 0"/><mass value="1"/><inertia ixx="1" ixy="0" ixz="0" iyy="1" iyz="0" izz="1"/></inertial>
@@ -116,5 +107,4 @@
     <limit lower="0.0" upper="0.0" effort="1e9" velocity="0.0"/>
   </joint>
-  <!-- Front LEFT (idler) -->
   <link name="fl_1">
     <inertial>
@@ -130,5 +120,5 @@
       <origin xyz="0 0 0" rpy="0 0 0"/>
       <geometry>
-        <mesh filename="${pkg_share}/meshes/wheel.dae" scale="0.5 0.5 0.5"/>
+        <mesh filename="package://alphabot_description/meshes/wheel.dae" scale="0.5 0.5 0.5"/>
       </geometry>
     </visual>
@@ -140,5 +130,4 @@
     <axis xyz="1 0 0"/>
   </joint>
-  <!-- Front RIGHT (idler) -->
   <link name="fr_1">
     <inertial>
@@ -154,5 +143,5 @@
       <origin xyz="0 0 0" rpy="0 0 0"/>
       <geometry>
-        <mesh filename="${pkg_share}/meshes/wheel.dae" scale="0.5 0.5 0.5"/>
+        <mesh filename="package://alphabot_description/meshes/wheel.dae" scale="0.5 0.5 0.5"/>
       </geometry>
     </visual>
@@ -164,5 +153,4 @@
     <axis xyz="1 0 0"/>
   </joint>
-  <!-- ================== LiDAR & Lift ================== -->
   <link name="lidar_link">
     <inertial><origin xyz="0 0 0"/><mass value="0.5"/><inertia ixx="0.001" ixy="0" ixz="0" iyy="0.001" iyz="0" izz="0.001"/></inertial>
@@ -180,5 +168,5 @@
       <origin xyz="0 0 0.1" rpy="0 0 0"/>
       <geometry>
-        <mesh filename="${pkg_share}/meshes/platform.dae" scale="0.5 0.5 0.5"/>
+        <mesh filename="package://alphabot_description/meshes/platform.dae" scale="0.5 0.5 0.5"/>
       </geometry>
     </visual>
@@ -193,5 +181,4 @@
     <child  link="lift_link"/>
   </joint>
-  <!-- ================== Camera frames ================== -->
   <link name="camera_mount_link">
     <inertial><origin xyz="0 0 0"/><mass value="0.1"/><inertia ixx="0.0001" ixy="0" ixz="0" iyy="0.0001" iyz="0" izz="0.0001"/></inertial>
@@ -214,5 +201,4 @@
     <child  link="camera_optical_frame"/>
   </joint>
-  <!-- ================== Gazebo materials/contacts ================== -->
   <gazebo reference="chassis_link"><selfCollide>true</selfCollide><mu1>0.2</mu1><mu2>0.2</mu2></gazebo>
   <gazebo reference="bl_1"><mu1>1e6</mu1><mu2>1e6</mu2></gazebo>
@@ -221,5 +207,4 @@
   <gazebo reference="fr_1"><mu1>1e6</mu1><mu2>1e6</mu2></gazebo>
   <gazebo reference="lift_link"><mu1>1e6</mu1><mu2>1e5</mu2><kp>1e5</kp><kd>1</kd><maxVel>0.01</maxVel><minDepth>0.001</minDepth></gazebo>
-  <!-- ================== Gazebo: LIDAR ================== -->
   <gazebo reference="lidar_link">
     <sensor name="lidar" type="ray">
