Commit message: Added depth

File: ALPHA_BOT/alphabot_description/urdf/alphabot.urdf.xacro (robot description, xacro)
@@ -1,8 +1,10 @@
 <?xml version="1.0"?>
 <robot name="alphabot" xmlns:xacro="http://www.ros.org/wiki/xacro">
+  <!-- Args / properties -->
   <xacro:property name="use_gazebo_camera" value="true"/>
   <xacro:property name="cmd_vel_topic"     value="/amazon_robot/cmd_vel"/>
   <xacro:property name="odom_topic"        value="/amazon_robot/odom"/>
   <xacro:property name="scan_topic"        value="/scan"/>
+  <!-- ================== Base frames ================== -->
   <link name="base_footprint"/>
   <link name="base_link"/>
@@ -12,4 +14,5 @@
     <origin xyz="0 0 0.072" rpy="0 0 0"/>
   </joint>
+  <!-- ================== Chassis ================== -->
   <link name="chassis_link">
     <inertial>
@@ -37,6 +40,5 @@
   </joint>
   <!-- ================== Wheels ================== -->
-  <!-- Shared wheel params: radius=0.072, width=0.06; we orient cyl axis along X (rpy 0 1.5708 0) -->
-  <!-- Rear LEFT (drive) -->
+  <!-- Rear LEFT -->
   <link name="bl_1">
     <inertial>
@@ -63,4 +65,5 @@
     <dynamics friction="12.0316061502"/>
   </joint>
+  <!-- Rear RIGHT -->
   <link name="br_1">
     <inertial>
@@ -107,4 +110,5 @@
     <limit lower="0.0" upper="0.0" effort="1e9" velocity="0.0"/>
   </joint>
+  <!-- Front wheels -->
   <link name="fl_1">
     <inertial>
@@ -153,4 +157,5 @@
     <axis xyz="1 0 0"/>
   </joint>
+  <!-- ================== LiDAR & Lift ================== -->
   <link name="lidar_link">
     <inertial><origin xyz="0 0 0"/><mass value="0.5"/><inertia ixx="0.001" ixy="0" ixz="0" iyy="0.001" iyz="0" izz="0.001"/></inertial>
@@ -181,24 +186,78 @@
     <child  link="lift_link"/>
   </joint>
-  <link name="camera_mount_link">
-    <inertial><origin xyz="0 0 0"/><mass value="0.1"/><inertia ixx="0.0001" ixy="0" ixz="0" iyy="0.0001" iyz="0" izz="0.0001"/></inertial>
-  </link>
-  <joint name="camera_mount_joint" type="fixed">
-    <origin xyz="0 0.45 0.09" rpy="0 0 0"/>
+  <!-- ================== RealSense D435 ================== -->
+  <link name="realsense_link">
+    <inertial>
+      <origin xyz="0 0 0" rpy="1.57 0 1.57"/>
+      <mass value="0.0615752"/>
+      <inertia ixx="9.108e-05" ixy="0" ixz="0" iyy="2.51e-06" iyz="0" izz="8.931e-05"/>
+    </inertial>
+    <visual name="visual">
+      <origin xyz="0 0 0" rpy="1.57 0 1.57"/>
+      <geometry>
+        <mesh filename="package://alphabot_description/meshes/RealSense_D435/realsense.dae"/>
+      </geometry>
+      <material>
+        <script>
+          <uri>package://alphabot_description/RealSense_D435/materials/scripts/</uri>
+          <uri>package://alphabot_description/RealSense_D435/materials/textures/</uri>
+          <name>UrbanTile/RealSense_Diffuse</name>
+        </script>
+      </material>
+    </visual>
+    <collision name="collision">
+      <origin xyz="0 0 0" rpy="1.57 0 1.57"/>
+      <geometry>
+        <mesh filename="package://alphabot_description/meshes/RealSense_D435/realsense.dae"/>
+      </geometry>
+    </collision>
+  </link>
+  <!-- Mount pose -->
+  <joint name="realsense_joint" type="fixed">
+    <origin xyz="0.071927 -1.097241 1.312280" rpy="1.799222 0 1.57"/>
     <parent link="base_link"/>
-    <child  link="camera_mount_link"/>
-  </joint>
-  <link name="camera_link"/>
-  <joint name="camera_joint" type="fixed">
-    <parent link="camera_mount_link"/>
-    <child  link="camera_link"/>
+    <child  link="realsense_link"/>
+  </joint>
+  <!-- Depth frames only (REP 105) -->
+  <link name="realsense_depth_frame"/>
+  <joint name="realsense_depth_frame_joint" type="fixed">
     <origin xyz="0 0 0" rpy="0 0 0"/>
-  </joint>
-  <link name="camera_optical_frame"/>
-  <joint name="camera_optical_joint" type="fixed">
+    <parent link="realsense_link"/><child link="realsense_depth_frame"/>
+  </joint>
+  <link name="realsense_depth_optical_frame"/>
+  <joint name="realsense_depth_optical_joint" type="fixed">
     <origin xyz="0 0 0" rpy="0 -1.57079632679 3.14159265359"/>
-    <parent link="camera_link"/>
-    <child  link="camera_optical_frame"/>
-  </joint>
+    <parent link="realsense_depth_frame"/><child link="realsense_depth_optical_frame"/>
+  </joint>
+  <!-- ================== Gazebo sensor: SINGLE depth camera with image+info+pointcloud ================== -->
+  <gazebo reference="realsense_link">
+    <sensor name="realsense_depth_camera" type="depth">
+      <always_on>1</always_on>
+      <update_rate>30</update_rate>
+      <visualize>0</visualize>
+      <pose>0 0 0 0 0 -1.5708</pose>
+      <camera name="depth_camera">
+        <horizontal_fov>1.0472</horizontal_fov>
+        <image>
+          <width>640</width>
+          <height>480</height>
+          <format>B8G8R8</format>
+        </image>
+        <clip><near>0.01</near><far>10</far></clip>
+      </camera>
+      <plugin name="realsense_depth_plugin" filename="libgazebo_ros_camera.so">
+        <ros>
+          <remapping>image_raw:=/realsense_depth_camera/depth/image_raw</remapping>
+          <remapping>camera_info:=/realsense_depth_camera/depth/camera_info</remapping>
+          <remapping>points:=/realsense_depth_camera/points</remapping>
+        </ros>
+        <frame_name>realsense_depth_optical_frame</frame_name>
+        <output_pointcloud>true</output_pointcloud>
+        <pointCloudCutoff>0.01</pointCloudCutoff>
+        <pointCloudCutoffMax>10.0</pointCloudCutoffMax>
+      </plugin>
+    </sensor>
+  </gazebo>
+  <!-- ================== Gazebo materials/contacts ================== -->
   <gazebo reference="chassis_link"><selfCollide>true</selfCollide><mu1>0.2</mu1><mu2>0.2</mu2></gazebo>
   <gazebo reference="bl_1"><mu1>1e6</mu1><mu2>1e6</mu2></gazebo>
@@ -207,4 +266,5 @@
   <gazebo reference="fr_1"><mu1>1e6</mu1><mu2>1e6</mu2></gazebo>
   <gazebo reference="lift_link"><mu1>1e6</mu1><mu2>1e5</mu2><kp>1e5</kp><kd>1</kd><maxVel>0.01</maxVel><minDepth>0.001</minDepth></gazebo>
+  <!-- ================== LIDAR (unchanged) ================== -->
   <gazebo reference="lidar_link">
     <sensor name="lidar" type="ray">
@@ -221,19 +281,9 @@
           </horizontal>
         </scan>
-        <range>
-          <min>0.12</min>
-          <max>30.0</max>
-          <resolution>0.01</resolution>
-        </range>
-        <noise>
-          <type>gaussian</type>
-          <mean>0.0</mean>
-          <stddev>0.01</stddev>
-        </noise>
+        <range><min>0.12</min><max>20.0</max><resolution>0.01</resolution></range>
+        <noise><type>gaussian</type><mean>0.0</mean><stddev>0.01</stddev></noise>
       </ray>
       <plugin name="gazebo_ros_ray_sensor" filename="libgazebo_ros_ray_sensor.so">
-        <ros>
-          <remapping>~/out:=$(arg scan_topic)</remapping>
-        </ros>
+        <ros><remapping>~/out:=$(arg scan_topic)</remapping></ros>
         <output_type>sensor_msgs/LaserScan</output_type>
         <frame_name>lidar_link</frame_name>
@@ -241,32 +291,8 @@
     </sensor>
   </gazebo>
-  <!-- ================== Gazebo: camera (optional) ================== -->
-  <xacro:if value="$(arg use_gazebo_camera)">
-    <gazebo reference="camera_link">
-      <sensor name="sim_camera" type="camera">
-        <update_rate>30</update_rate>
-        <camera>
-          <horizontal_fov>1.39626</horizontal_fov>
-          <image>
-            <width>640</width>
-            <height>480</height>
-            <format>R8G8B8</format>
-          </image>
-          <clip><near>0.02</near><far>50.0</far></clip>
-        </camera>
-        <plugin name="gazebo_ros_camera" filename="libgazebo_ros_camera.so">
-          <ros>
-            <remapping>image_raw:=/camera/image_raw</remapping>
-            <remapping>camera_info:=/camera/camera_info</remapping>
-            <frame_name>camera_optical_frame</frame_name>
-          </ros>
-        </plugin>
-      </sensor>
-    </gazebo>
-  </xacro:if>
-  <!-- ================== Gazebo: joint state publisher ================== -->
+  <!-- ================== Gazebo: joint states + diff drive ================== -->
   <gazebo>
     <plugin name="joint_state_publisher" filename="libgazebo_ros_joint_state_publisher.so">
-      <update_rate>50</update_rate>
+      <update_rate>100</update_rate>
       <joint_name>bl_axle</joint_name>
       <joint_name>br_axle</joint_name>
@@ -277,5 +303,4 @@
     </plugin>
   </gazebo>
-  <!-- ================== Gazebo: differential drive ================== -->
   <gazebo>
     <plugin name="diff_drive" filename="libgazebo_ros_diff_drive.so">
@@ -296,5 +321,4 @@
       <odometry_frame>odom</odometry_frame>
       <robot_base_frame>base_footprint</robot_base_frame>
-      <!-- 0 = ENCODER, 1 = WORLD -->
       <odometry_source>0</odometry_source>
     </plugin>

Commit message: backup

File: ALPHA_BOT/alphabot_description/urdf/alphabot.urdf.xacro (robot description, xacro)
@@ -187,48 +187,45 @@
   </joint>
   <!-- ================== RealSense D435 ================== -->
+  <!-- Camera body (mesh orientation baked in visuals; TF comes from joints) -->
   <link name="realsense_link">
     <inertial>
-      <origin xyz="0 0 0" rpy="1.57 0 1.57"/>
+      <origin xyz="0 0 0" rpy="0 0 0"/>
       <mass value="0.0615752"/>
       <inertia ixx="9.108e-05" ixy="0" ixz="0" iyy="2.51e-06" iyz="0" izz="8.931e-05"/>
     </inertial>
     <visual name="visual">
-      <origin xyz="0 0 0" rpy="1.57 0 1.57"/>
-      <geometry>
-        <mesh filename="package://alphabot_description/meshes/RealSense_D435/realsense.dae"/>
-      </geometry>
-      <material>
-        <script>
-          <uri>package://alphabot_description/RealSense_D435/materials/scripts/</uri>
-          <uri>package://alphabot_description/RealSense_D435/materials/textures/</uri>
-          <name>UrbanTile/RealSense_Diffuse</name>
-        </script>
-      </material>
+      <origin xyz="0 0 0" rpy="0 0 0"/>
+      <geometry>
+        <mesh filename="package://alphabot_description/meshes/RealSense_D435/meshes/realsense.dae"/>
+      </geometry>
     </visual>
     <collision name="collision">
-      <origin xyz="0 0 0" rpy="1.57 0 1.57"/>
-      <geometry>
-        <mesh filename="package://alphabot_description/meshes/RealSense_D435/realsense.dae"/>
-      </geometry>
-    </collision>
-  </link>
-  <!-- Mount pose -->
+      <origin xyz="0 0 0" rpy="0 0 0"/>
+      <geometry>
+        <mesh filename="package://alphabot_description/meshes/RealSense_D435/meshes/realsense.dae"/>
+      </geometry>
+    </collision>
+  </link>
+  <!-- Mount pose: match your original SDF orientation, new xyz (0 0.45 0.19) -->
   <joint name="realsense_joint" type="fixed">
-    <origin xyz="0.071927 -1.097241 1.312280" rpy="1.799222 0 1.57"/>
+    <origin xyz="0 0.45 0.19" rpy="0 0 1.57"/>
     <parent link="base_link"/>
     <child  link="realsense_link"/>
   </joint>
-  <!-- Depth frames only (REP 105) -->
+  <!-- Depth frames (REP-105) -->
   <link name="realsense_depth_frame"/>
   <joint name="realsense_depth_frame_joint" type="fixed">
-    <origin xyz="0 0 0" rpy="0 0 0"/>
-    <parent link="realsense_link"/><child link="realsense_depth_frame"/>
+    <origin xyz="0 0 0" rpy="-1.57 0 3.14"/>
+    <parent link="realsense_link"/>
+    <child  link="realsense_depth_frame"/>
   </joint>
   <link name="realsense_depth_optical_frame"/>
   <joint name="realsense_depth_optical_joint" type="fixed">
-    <origin xyz="0 0 0" rpy="0 -1.57079632679 3.14159265359"/>
-    <parent link="realsense_depth_frame"/><child link="realsense_depth_optical_frame"/>
-  </joint>
-  <!-- ================== Gazebo sensor: SINGLE depth camera with image+info+pointcloud ================== -->
+    <!-- X right, Y down, Z forward -->
+    <origin xyz="0 0 0" rpy="-1.57 -1.57 1.57"/>
+    <parent link="realsense_depth_frame"/>
+    <child  link="realsense_depth_optical_frame"/>
+  </joint>
+  <!-- Gazebo sensor: single depth cam (image + info + point cloud) -->
   <gazebo reference="realsense_link">
     <sensor name="realsense_depth_camera" type="depth">
@@ -236,12 +233,9 @@
       <update_rate>30</update_rate>
       <visualize>0</visualize>
-      <pose>0 0 0 0 0 -1.5708</pose>
+      <!-- No extra rotation; joint above defines the body orientation -->
+      <pose>0 0 0 0 0 0</pose>
       <camera name="depth_camera">
         <horizontal_fov>1.0472</horizontal_fov>
-        <image>
-          <width>640</width>
-          <height>480</height>
-          <format>B8G8R8</format>
-        </image>
+        <image><width>640</width><height>480</height><format>B8G8R8</format></image>
         <clip><near>0.01</near><far>10</far></clip>
       </camera>

Commit message: Added two storied building

File: ALPHA_BOT/alphabot_description/urdf/alphabot.urdf.xacro (robot description, xacro)
@@ -190,10 +190,10 @@
   <link name="realsense_link">
     <inertial>
-      <origin xyz="0 0 0" rpy="0 0 0"/>
+      <origin xyz="0 0 0" rpy="0 0 1.57"/>
       <mass value="0.0615752"/>
       <inertia ixx="9.108e-05" ixy="0" ixz="0" iyy="2.51e-06" iyz="0" izz="8.931e-05"/>
     </inertial>
     <visual name="visual">
-      <origin xyz="0 0 0" rpy="0 0 0"/>
+      <origin xyz="0 0 0" rpy="0 0 1.57"/>
       <geometry>
         <mesh filename="package://alphabot_description/meshes/RealSense_D435/meshes/realsense.dae"/>
@@ -201,5 +201,5 @@
     </visual>
     <collision name="collision">
-      <origin xyz="0 0 0" rpy="0 0 0"/>
+     <origin xyz="0 0 0" rpy="0 0 1.57"/>
       <geometry>
         <mesh filename="package://alphabot_description/meshes/RealSense_D435/meshes/realsense.dae"/>

Commit message: Refactor bringup and description for mobile manipulator with linear guide
- Updated bringup_gazebo.launch.py to include environment variable settings for GAZEBO_MODEL_PATH and GAZEBO_PLUGIN_PATH.
- Modified CMakeLists.txt in alphabot_description and elevator_plugin to include environment hooks for Gazebo paths.
- Added new environment hook files for gazebo_model_path and gazebo_plugin_path.
- Refactored URDF files to use xacro arguments for better configurability.
- Adjusted camera pose in no_roof_small_warehouse.world for improved visibility.
- Enhanced the mobile manipulator bringup launch file to include new linear guide components and controllers.
- Added new meshes for base and vertical column to the mobile manipulator package.
- Created a new URDF file for the linear guide with appropriate joints and plugins.
- Updated package.xml to reflect new dependencies and descriptions.

File: ALPHA_BOT/alphabot_description/urdf/alphabot.urdf.xacro (robot description, xacro)
@@ -2,8 +2,8 @@
 <robot name="alphabot" xmlns:xacro="http://www.ros.org/wiki/xacro">
   <!-- Args / properties -->
-  <xacro:property name="use_gazebo_camera" value="true"/>
-  <xacro:property name="cmd_vel_topic"     value="/amazon_robot/cmd_vel"/>
-  <xacro:property name="odom_topic"        value="/amazon_robot/odom"/>
-  <xacro:property name="scan_topic"        value="/scan"/>
+  <xacro:arg name="scan_topic" default="/scan"/>
+  <xacro:arg name="cmd_vel_topic" default="/amazon_robot/cmd_vel"/>
+  <xacro:arg name="odom_topic" default="/amazon_robot/odom"/>
+  <xacro:arg name="use_gazebo_camera" default="true"/>
   <!-- ================== Base frames ================== -->
   <link name="base_footprint"/>

Commit message: Refactor mobile manipulator launch files and configurations; integrate linear guide and arm controllers

File: ALPHA_BOT/alphabot_description/urdf/alphabot.urdf.xacro (robot description, xacro)
@@ -1,15 +1,13 @@
 <?xml version="1.0"?>
 <robot name="alphabot" xmlns:xacro="http://www.ros.org/wiki/xacro">
-  <!-- Args / properties -->
   <xacro:arg name="scan_topic" default="/scan"/>
   <xacro:arg name="cmd_vel_topic" default="/amazon_robot/cmd_vel"/>
   <xacro:arg name="odom_topic" default="/amazon_robot/odom"/>
   <xacro:arg name="use_gazebo_camera" default="true"/>
-  <!-- ================== Base frames ================== -->
   <link name="base_footprint"/>
-  <link name="base_link"/>
+  <link name="link_base"/>
   <joint name="base_joint" type="fixed">
     <parent link="base_footprint"/>
-    <child  link="base_link"/>
+    <child  link="link_base"/>
     <origin xyz="0 0 0.072" rpy="0 0 0"/>
   </joint>
@@ -35,5 +33,5 @@
   </link>
   <joint name="chassis_link_joint" type="fixed">
-    <parent link="base_link"/>
+    <parent link="link_base"/>
     <child  link="chassis_link"/>
     <origin xyz="0 0 0" rpy="0 0 0"/>
@@ -165,5 +163,5 @@
   <joint name="lidar_joint" type="fixed">
     <origin xyz="0 0 0.18" rpy="0 0 0"/>
-    <parent link="base_link"/>
+    <parent link="link_base"/>
     <child  link="lidar_link"/>
   </joint>
@@ -210,5 +208,5 @@
   <joint name="realsense_joint" type="fixed">
     <origin xyz="0 0.45 0.19" rpy="0 0 1.57"/>
-    <parent link="base_link"/>
+    <parent link="link_base"/>
     <child  link="realsense_link"/>
   </joint>
@@ -264,17 +262,17 @@
     <sensor name="lidar" type="ray">
       <always_on>true</always_on>
-      <update_rate>20</update_rate>
+      <update_rate>30</update_rate>
       <visualize>true</visualize>
       <ray>
         <scan>
           <horizontal>
-            <samples>720</samples>
+            <samples>361</samples>
             <resolution>1</resolution>
-            <min_angle>-3.14159265</min_angle>
+            <min_angle>0</min_angle>
             <max_angle>3.14159265</max_angle>
           </horizontal>
         </scan>
-        <range><min>0.12</min><max>20.0</max><resolution>0.01</resolution></range>
-        <noise><type>gaussian</type><mean>0.0</mean><stddev>0.01</stddev></noise>
+        <range><min>0.55</min><max>16.0</max><resolution>0.01</resolution></range>
+        <noise><type>gaussian</type><mean>0.0</mean><stddev>0.0</stddev></noise>
       </ray>
       <plugin name="gazebo_ros_ray_sensor" filename="libgazebo_ros_ray_sensor.so">
@@ -286,5 +284,5 @@
   </gazebo>
   <!-- ================== Gazebo: joint states + diff drive ================== -->
-  <gazebo>
+  <!-- <gazebo>
     <plugin name="joint_state_publisher" filename="libgazebo_ros_joint_state_publisher.so">
       <update_rate>100</update_rate>
@@ -317,4 +315,4 @@
       <odometry_source>0</odometry_source>
     </plugin>
-  </gazebo>
+  </gazebo> -->
 </robot>
