Commit message: Refactor mobile manipulator configuration and integration; update controllers and URDF files for improved functionality

File: ALPHA_BOT/alphabot_description/urdf/alphabot.urdf.xacro (robot description, xacro)
@@ -12,5 +12,4 @@
     <origin xyz="0 0 0.072" rpy="0 0 0"/>
   </joint>
-  <!-- ================== Chassis ================== -->
   <link name="chassis_link">
     <inertial>
@@ -37,6 +36,4 @@
     <origin xyz="0 0 0" rpy="0 0 0"/>
   </joint>
-  <!-- ================== Wheels ================== -->
-  <!-- Rear LEFT -->
   <link name="bl_1">
     <inertial>
@@ -63,5 +60,4 @@
     <dynamics friction="12.0316061502"/>
   </joint>
-  <!-- Rear RIGHT -->
   <link name="br_1">
     <inertial>
@@ -108,5 +104,4 @@
     <limit lower="0.0" upper="0.0" effort="1e9" velocity="0.0"/>
   </joint>
-  <!-- Front wheels -->
   <link name="fl_1">
     <inertial>
@@ -155,5 +150,4 @@
     <axis xyz="1 0 0"/>
   </joint>
-  <!-- ================== LiDAR & Lift ================== -->
   <link name="lidar_link">
     <inertial><origin xyz="0 0 0"/><mass value="0.5"/><inertia ixx="0.001" ixy="0" ixz="0" iyy="0.001" iyz="0" izz="0.001"/></inertial>
@@ -184,6 +178,4 @@
     <child  link="lift_link"/>
   </joint>
-  <!-- ================== RealSense D435 ================== -->
-  <!-- Camera body (mesh orientation baked in visuals; TF comes from joints) -->
   <link name="realsense_link">
     <inertial>
@@ -205,5 +197,4 @@
     </collision>
   </link>
-  <!-- Mount pose: match your original SDF orientation, new xyz (0 0.45 0.19) -->
   <joint name="realsense_joint" type="fixed">
     <origin xyz="0 0.45 0.19" rpy="0 0 1.57"/>
@@ -211,5 +202,4 @@
     <child  link="realsense_link"/>
   </joint>
-  <!-- Depth frames (REP-105) -->
   <link name="realsense_depth_frame"/>
   <joint name="realsense_depth_frame_joint" type="fixed">
@@ -220,10 +210,8 @@
   <link name="realsense_depth_optical_frame"/>
   <joint name="realsense_depth_optical_joint" type="fixed">
-    <!-- X right, Y down, Z forward -->
     <origin xyz="0 0 0" rpy="-1.57 -1.57 1.57"/>
     <parent link="realsense_depth_frame"/>
     <child  link="realsense_depth_optical_frame"/>
   </joint>
-  <!-- Gazebo sensor: single depth cam (image + info + point cloud) -->
   <gazebo reference="realsense_link">
     <sensor name="realsense_depth_camera" type="depth">
@@ -231,5 +219,4 @@
       <update_rate>30</update_rate>
       <visualize>0</visualize>
-      <!-- No extra rotation; joint above defines the body orientation -->
       <pose>0 0 0 0 0 0</pose>
       <camera name="depth_camera">
@@ -251,5 +238,4 @@
     </sensor>
   </gazebo>
-  <!-- ================== Gazebo materials/contacts ================== -->
   <gazebo reference="chassis_link"><selfCollide>true</selfCollide><mu1>0.2</mu1><mu2>0.2</mu2></gazebo>
   <gazebo reference="bl_1"><mu1>1e6</mu1><mu2>1e6</mu2></gazebo>
@@ -258,5 +244,4 @@
   <gazebo reference="fr_1"><mu1>1e6</mu1><mu2>1e6</mu2></gazebo>
   <gazebo reference="lift_link"><mu1>1e6</mu1><mu2>1e5</mu2><kp>1e5</kp><kd>1</kd><maxVel>0.01</maxVel><minDepth>0.001</minDepth></gazebo>
-  <!-- ================== LIDAR (unchanged) ================== -->
   <gazebo reference="lidar_link">
     <sensor name="lidar" type="ray">
@@ -283,5 +268,4 @@
     </sensor>
   </gazebo>
-  <!-- ================== Gazebo: joint states + diff drive ================== -->
   <!-- <gazebo>
     <plugin name="joint_state_publisher" filename="libgazebo_ros_joint_state_publisher.so">

File: MOBILE_MANIPULATOR/mobile_manipulator_description/urdf/linear_guide.xacro (robot description, xacro)
@@ -1,11 +1,10 @@
 <?xml version="1.0"?>
 <robot name="linear_guide" xmlns:xacro="http://ros.org/wiki/xacro">
-  <!-- Vertical column -->
   <link name="column">
     <visual>
       <geometry>
-        <box size="0.1 0.1 1.0"/> <!-- 10cm x 10cm, 1m tall -->
+        <box size="0.1 0.1 1.0"/>
       </geometry>
-      <origin xyz="0 0 0.5" rpy="0 0 0"/> <!-- column rests on ground -->
+      <origin xyz="0 0 0.5" rpy="0 0 0"/>
       <material name="grey">
         <color rgba="0.5 0.5 0.5 1.0"/>
@@ -23,11 +22,10 @@
     </inertial>
   </link>
-  <!-- Slider/Base (larger, sits at bottom) -->
   <link name="slider">
     <visual>
       <geometry>
-        <box size="0.6 0.6 0.1"/> <!-- 40cm x 40cm, 10cm thick -->
+        <box size="0.6 0.6 0.1"/>
       </geometry>
-      <origin xyz="0 -0.25 0.05" rpy="0 0 0"/> <!-- sits on ground -->
+      <origin xyz="0 -0.25 0.05" rpy="0 0 0"/>
       <material name="blue">
         <color rgba="0.1 0.1 0.8 1.0"/>
@@ -38,5 +36,5 @@
         <box size="0.6 0.6 0.1"/>
       </geometry>
-      <origin xyz="0 0 0.05" rpy="0 0 0"/>
+      <origin xyz="0 -0.25 0.05" rpy="0 0 0"/>
     </collision>
     <inertial>
@@ -45,27 +43,10 @@
     </inertial>
   </link>
-  <!-- Prismatic Joint (slider moves up along Z from ground) -->
   <joint name="slider_joint" type="prismatic">
     <parent link="column"/>
     <child link="slider"/>
-    <origin xyz="0 0 0" rpy="0 0 0"/> <!-- start at bottom -->
-    <axis xyz="0 0 1"/> <!-- move along Z-axis -->
+    <origin xyz="0 0 0" rpy="0 0 0"/>
+    <axis xyz="0 0 1"/>
     <limit lower="0.0" upper="0.9" effort="200" velocity="0.3"/>
   </joint>
-<!--
-  <gazebo>
-  <plugin name="gazebo_ros_control" filename="libgazebo_ros_control.so"/>
-</gazebo>
-<gazebo reference="slider_joint">
-  <plugin name="slider_joint_position_controller" filename="libgazebo_ros_joint_position_controller.so">
-    <joint>slider_joint</joint>
-    <topic>slider_joint_position_controller/command</topic>
-    <pid>
-      <p>100.0</p>
-      <i>0.01</i>
-      <d>10.0</d>
-    </pid>
-  </plugin>
-</gazebo>
- -->
 </robot>

File: MOBILE_MANIPULATOR/mobile_manipulator_description/urdf/mobile_manipulator.urdf.xacro (robot description, xacro)
@@ -1,25 +1,16 @@
 <?xml version="1.0"?>
 <robot name="mobile_manipulator" xmlns:xacro="http://www.ros.org/wiki/xacro">
-  <!-- ================== INCLUDE SUBMODULES ================== -->
-  <!-- Mobile robot -->
   <xacro:include filename="$(find alphabot_description)/urdf/alphabot.urdf.xacro"/>
-  <!-- Linear guide -->
   <xacro:include filename="$(find mobile_manipulator_description)/urdf/linear_guide.xacro"/>
-  <!-- Realman RM-75 Arm -->
   <xacro:include filename="$(find rm_description)/urdf/rm_75_gazebo.urdf"/>
   <xacro:include filename="$(find mobile_manipulator_description)/urdf/mobile_manipulator_ros_contol.xacro"/>
-  <!-- ================== INTEGRATION ================== -->
-  <!-- 1. Mount linear guide column to mobile robot chassis -->
   <joint name="chassis_to_column" type="fixed">
-    <parent link="chassis_link"/>  <!-- from alphabot -->
-    <child  link="column"/>        <!-- from linear guide -->
-    <!-- Adjust placement of linear guide relative to robot base -->
+    <parent link="chassis_link"/>
+    <child  link="column"/>
     <origin xyz="0 0 0.33" rpy="0 0 0"/>
   </joint>
-  <!-- 2. Prismatic joint already exists: column ↔ slider -->
-  <!-- 3. Mount robotic arm base_link to slider -->
   <joint name="slider_to_arm_base" type="fixed">
-    <parent link="slider"/>        <!-- moving part of linear guide -->
-    <child  link="base_link"/>     <!-- arm base_link from rm_75 -->
+    <parent link="slider"/>
+    <child  link="base_link"/>
     <origin xyz="0 -0.25 0.13" rpy="0 0 0"/>
   </joint>
@@ -31,8 +22,6 @@
   <gazebo>
     <plugin filename="libgazebo_ros2_control.so" name="gazebo_ros2_control">
-      <!-- robot_description param is provided by robot_state_publisher -->
       <robot_param>robot_description</robot_param>
       <robot_param_node>robot_state_publisher</robot_param_node>
-      <!-- point to your controller config -->
       <parameters>$(find mobile_manipulator_control)/config/controllers.yaml</parameters>
     </plugin>

File: MOBILE_MANIPULATOR/mobile_manipulator_description/urdf/mobile_manipulator_ros_contol.xacro (robot description, xacro)
@@ -1,21 +1,18 @@
 <?xml version="1.0"?>
 <robot name="mobile_manipulator" xmlns:xacro="http://www.ros.org/wiki/xacro">
-  <!-- ros2_control hardware and joints -->
   <ros2_control name="GazeboSystem" type="system">
     <hardware>
       <plugin>gazebo_ros2_control/GazeboSystem</plugin>
     </hardware>
-    <!-- Mobile base wheels -->
-    <joint name="bl_1">
+    <joint name="bl_axle">
       <command_interface name="velocity"/>
+      <state_interface name="velocity"/>
       <state_interface name="position"/>
+    </joint>
+    <joint name="br_axle">
+      <command_interface name="velocity"/>
       <state_interface name="velocity"/>
+      <state_interface name="position"/>
     </joint>
-    <joint name="br_1">
-      <command_interface name="velocity"/>
-      <state_interface name="position"/>
-      <state_interface name="velocity"/>
-    </joint>
-    <!-- Slider joint -->
     <joint name="slider_joint">
       <command_interface name="position"/>
@@ -23,5 +20,4 @@
       <state_interface name="velocity"/>
     </joint>
-    <!-- Arm joints -->
     <joint name="joint1">
       <command_interface name="position"/>
@@ -60,3 +56,48 @@
     </joint>
   </ros2_control>
+    <transmission name="bl_axle_trans">
+    <type>transmission_interface/SimpleTransmission</type>
+    <joint name="bl_axle">
+        <hardwareInterface>hardware_interface/VelocityCommandInterface</hardwareInterface>
+    </joint>
+    <actuator name="bl_axle_motor">
+        <hardwareInterface>hardware_interface/VelocityCommandInterface</hardwareInterface>
+    </actuator>
+    </transmission>
+    <transmission name="br_axle_trans">
+    <type>transmission_interface/SimpleTransmission</type>
+    <joint name="br_axle">
+        <hardwareInterface>hardware_interface/VelocityCommandInterface</hardwareInterface>
+    </joint>
+    <actuator name="br_axle_motor">
+        <hardwareInterface>hardware_interface/VelocityCommandInterface</hardwareInterface>
+    </actuator>
+    </transmission>
+  <transmission name="slider_trans">
+    <type>transmission_interface/SimpleTransmission</type>
+    <joint name="slider_joint">
+      <hardwareInterface>hardware_interface/PositionCommandInterface</hardwareInterface>
+    </joint>
+    <actuator name="slider_motor">
+      <hardwareInterface>hardware_interface/PositionCommandInterface</hardwareInterface>
+    </actuator>
+  </transmission>
+  <xacro:macro name="arm_transmission" params="joint_name">
+    <transmission name="${joint_name}_trans">
+      <type>transmission_interface/SimpleTransmission</type>
+      <joint name="${joint_name}">
+        <hardwareInterface>hardware_interface/PositionCommandInterface</hardwareInterface>
+      </joint>
+      <actuator name="${joint_name}_motor">
+        <hardwareInterface>hardware_interface/PositionCommandInterface</hardwareInterface>
+      </actuator>
+    </transmission>
+  </xacro:macro>
+  <xacro:arm_transmission joint_name="joint1"/>
+  <xacro:arm_transmission joint_name="joint2"/>
+  <xacro:arm_transmission joint_name="joint3"/>
+  <xacro:arm_transmission joint_name="joint4"/>
+  <xacro:arm_transmission joint_name="joint5"/>
+  <xacro:arm_transmission joint_name="joint6"/>
+  <xacro:arm_transmission joint_name="joint7"/>
 </robot>

Commit message: Refactor launch files and configurations for mobile manipulator; remove unused RViz arguments and update controller settings

File: ALPHA_BOT/alphabot_description/urdf/alphabot.urdf.xacro (robot description, xacro)
@@ -258,5 +258,5 @@
           </horizontal>
         </scan>
-        <range><min>0.55</min><max>16.0</max><resolution>0.01</resolution></range>
+        <range><min>0.10</min><max>16.0</max><resolution>0.01</resolution></range>
         <noise><type>gaussian</type><mean>0.0</mean><stddev>0.0</stddev></noise>
       </ray>
@@ -268,5 +268,5 @@
     </sensor>
   </gazebo>
-  <!-- <gazebo>
+  <gazebo>
     <plugin name="joint_state_publisher" filename="libgazebo_ros_joint_state_publisher.so">
       <update_rate>100</update_rate>
@@ -299,4 +299,4 @@
       <odometry_source>0</odometry_source>
     </plugin>
-  </gazebo> -->
+  </gazebo>
 </robot>

File: MOBILE_MANIPULATOR/mobile_manipulator_description/urdf/mobile_manipulator.urdf.xacro (robot description, xacro)
@@ -15,9 +15,10 @@
     <origin xyz="0 -0.25 0.13" rpy="0 0 0"/>
   </joint>
+<!--
   <link name="world"/>
   <joint name="world_to_robot" type="fixed">
     <parent link="world"/>
     <child link="base_footprint"/>
-  </joint>
+  </joint> -->
   <gazebo>
     <plugin filename="libgazebo_ros2_control.so" name="gazebo_ros2_control">

File: MOBILE_MANIPULATOR/mobile_manipulator_description/urdf/mobile_manipulator_ros_contol.xacro (robot description, xacro)
@@ -5,14 +5,4 @@
       <plugin>gazebo_ros2_control/GazeboSystem</plugin>
     </hardware>
-    <joint name="bl_axle">
-      <command_interface name="velocity"/>
-      <state_interface name="velocity"/>
-      <state_interface name="position"/>
-    </joint>
-    <joint name="br_axle">
-      <command_interface name="velocity"/>
-      <state_interface name="velocity"/>
-      <state_interface name="position"/>
-    </joint>
     <joint name="slider_joint">
       <command_interface name="position"/>
@@ -56,22 +46,4 @@
     </joint>
   </ros2_control>
-    <transmission name="bl_axle_trans">
-    <type>transmission_interface/SimpleTransmission</type>
-    <joint name="bl_axle">
-        <hardwareInterface>hardware_interface/VelocityCommandInterface</hardwareInterface>
-    </joint>
-    <actuator name="bl_axle_motor">
-        <hardwareInterface>hardware_interface/VelocityCommandInterface</hardwareInterface>
-    </actuator>
-    </transmission>
-    <transmission name="br_axle_trans">
-    <type>transmission_interface/SimpleTransmission</type>
-    <joint name="br_axle">
-        <hardwareInterface>hardware_interface/VelocityCommandInterface</hardwareInterface>
-    </joint>
-    <actuator name="br_axle_motor">
-        <hardwareInterface>hardware_interface/VelocityCommandInterface</hardwareInterface>
-    </actuator>
-    </transmission>
   <transmission name="slider_trans">
     <type>transmission_interface/SimpleTransmission</type>

Commit message: Refactor navigation and SLAM launch files; update parameters for improved functionality, add behavior server, and enhance RViz integration for better visualization and control.

File: ALPHA_BOT/alphabot_description/urdf/alphabot.urdf.xacro (robot description, xacro)
@@ -169,6 +169,8 @@
     </visual>
     <collision>
-      <origin xyz="0 0 0" rpy="0 0 0"/>
-      <geometry><box size="0.2805 0.2 0.03"/></geometry>
+      <origin xyz="0 0 0.1" rpy="0 0 0"/>
+      <geometry>
+      <mesh filename="package://alphabot_description/meshes/platform.dae" scale="0.5 0.5 0.5"/>
+      </geometry>
     </collision>
   </link>
@@ -198,5 +200,5 @@
   </link>
   <joint name="realsense_joint" type="fixed">
-    <origin xyz="0 0.45 0.19" rpy="0 0 1.57"/>
+    <origin xyz="0 0.45 0.15" rpy="0 0 1.57"/>
     <parent link="link_base"/>
     <child  link="realsense_link"/>
@@ -245,22 +247,33 @@
   <gazebo reference="lift_link"><mu1>1e6</mu1><mu2>1e5</mu2><kp>1e5</kp><kd>1</kd><maxVel>0.01</maxVel><minDepth>0.001</minDepth></gazebo>
   <gazebo reference="lidar_link">
-    <sensor name="lidar" type="ray">
+    <sensor name="amr_lidar" type="ray">
       <always_on>true</always_on>
-      <update_rate>30</update_rate>
+      <update_rate>15</update_rate> <!-- 10-15 Hz like real sensors -->
       <visualize>true</visualize>
       <ray>
         <scan>
           <horizontal>
-            <samples>361</samples>
+            <samples>1080</samples>        <!-- 0.33° per beam -->
             <resolution>1</resolution>
-            <min_angle>0</min_angle>
+            <min_angle>-3.14159265</min_angle>
             <max_angle>3.14159265</max_angle>
           </horizontal>
         </scan>
-        <range><min>0.10</min><max>16.0</max><resolution>0.01</resolution></range>
-        <noise><type>gaussian</type><mean>0.0</mean><stddev>0.0</stddev></noise>
+        <range>
+          <min>0.12</min>       <!-- avoid robot self-collision -->
+          <max>25.0</max>       <!-- typical outdoor lidar range -->
+          <resolution>0.001</resolution>
+        </range>
+        <noise>
+          <type>gaussian</type>
+          <mean>0.0</mean>
+          <stddev>0.01</stddev>  <!-- 1 cm noise, realistic -->
+        </noise>
       </ray>
       <plugin name="gazebo_ros_ray_sensor" filename="libgazebo_ros_ray_sensor.so">
-        <ros><remapping>~/out:=$(arg scan_topic)</remapping></ros>
+        <ros>
+          <parameter name="use_sim_time" value="true"/>
+          <remapping>~/out:=/scan</remapping> <!-- topic published -->
+        </ros>
         <output_type>sensor_msgs/LaserScan</output_type>
         <frame_name>lidar_link</frame_name>
@@ -282,6 +295,7 @@
     <plugin name="diff_drive" filename="libgazebo_ros_diff_drive.so">
       <ros>
-        <remapping>cmd_vel:=$(arg cmd_vel_topic)</remapping>
-        <remapping>odom:=$(arg odom_topic)</remapping>
+      <parameter name="use_sim_time" value="true"/>
+      <remapping>cmd_vel:=/cmd_vel</remapping>
+      <remapping>odom:=/odom</remapping>
       </ros>
       <update_rate>100</update_rate>

Commit message: Chnage mesh files

File: ALPHA_BOT/alphabot_description/urdf/alphabot.urdf.xacro (robot description, xacro)
@@ -171,5 +171,5 @@
       <origin xyz="0 0 0.1" rpy="0 0 0"/>
       <geometry>
-      <mesh filename="package://alphabot_description/meshes/platform.dae" scale="0.5 0.5 0.5"/>
+      <mesh filename="package://alphabot_description/meshes/platform_collision.dae" scale="0.5 0.5 0.5"/>
       </geometry>
     </collision>
