Commit message: backup

File: ALPHA_BOT/alphabot_description/urdf/alphabot.urdf.xacro (robot description, xacro)
@@ -14,18 +14,18 @@
   <link name="chassis_link">
     <inertial>
-      <origin xyz="0 0 0" rpy="0 0 0"/>
+      <origin xyz="0 0 0" rpy="0 0 1.57"/>
       <mass value="1580"/>
       <inertia ixx="1997.86" ixy="0" ixz="0" iyy="442.769" iyz="62.5206" izz="2238.05"/>
     </inertial>
     <visual>
-      <origin xyz="0 0 0" rpy="0 0 0"/>
-      <geometry>
-        <mesh filename="package://alphabot_description/meshes/chassis.dae" scale="0.5 0.5 0.5"/>
+      <origin xyz="0 0 0" rpy="0 0 1.57"/>
+      <geometry>
+        <mesh filename="package://alphabot_description/meshes/chassy.dae" scale="1 1 1"/>
       </geometry>
     </visual>
     <collision>
-      <origin xyz="0 0 0" rpy="0 0 0"/>
-      <geometry>
-        <mesh filename="package://alphabot_description/meshes/chassis.dae" scale="0.5 0.5 0.5"/>
+      <origin xyz="0 0 0" rpy="0 0 1.57"/>
+      <geometry>
+        <mesh filename="package://alphabot_description/meshes/chassy.dae" scale="1 1 1"/>
       </geometry>
     </collision>
@@ -36,151 +36,129 @@
     <origin xyz="0 0 0" rpy="0 0 0"/>
   </joint>
-  <link name="bl_1">
-    <inertial>
+  <!-- ================= WHEELS (6 TOTAL, rotated Z) ================= -->
+  <!-- Front Left Trolley -->
+  <link name="front_left_wheel">
+    <collision><origin xyz="0 0 0" rpy="1.57 0 1.5708"/><geometry><sphere radius="0.0523"/></geometry></collision>
+    <inertial>
+      <origin xyz="0 0 0"/>
+      <mass value="0.1"/>
+      <inertia ixx="0.000144" iyy="0.000144" izz="0.000144"
+               ixy="0.0" ixz="0.0" iyz="0.0"/>
+    </inertial>
+  </link>
+  <joint name="front_left_wheel_joint" type="fixed">
+    <parent link="chassis_link"/>
+    <child link="front_left_wheel"/>
+    <origin xyz="0.40 0.27 -0.02" rpy="0 0 0"/>
+  </joint>
+  <!-- Front Right Trolley -->
+  <link name="front_right_wheel">
+    <collision><origin xyz="0 0 0" rpy="1.57 0 1.5708"/><geometry><sphere radius="0.0523"/></geometry></collision>
+    <inertial>
+      <origin xyz="0 0 0"/>
+      <mass value="0.1"/>
+      <inertia ixx="0.000144" iyy="0.000144" izz="0.000144"
+               ixy="0.0" ixz="0.0" iyz="0.0"/>
+    </inertial>
+  </link>
+  <joint name="front_right_wheel_joint" type="fixed">
+    <parent link="chassis_link"/>
+    <child link="front_right_wheel"/>
+    <origin xyz="0.40 -0.27 -0.02" rpy="0 0 0"/>
+  </joint>
+  <!-- Back Left Trolley -->
+  <link name="back_left_wheel">
+    <collision><origin xyz="0 0 0" rpy="1.57 0 1.5708"/><geometry><sphere radius="0.0523"/></geometry></collision>
+    <inertial>
+      <origin xyz="0 0 0"/>
+      <mass value="0.1"/>
+      <inertia ixx="0.000144" iyy="0.000144" izz="0.000144"
+               ixy="0.0" ixz="0.0" iyz="0.0"/>
+    </inertial>
+  </link>
+  <joint name="back_left_wheel_joint" type="fixed">
+    <parent link="chassis_link"/>
+    <child link="back_left_wheel"/>
+    <origin xyz="-0.40 0.27 -0.02" rpy="0 0 0"/>
+  </joint>
+  <!-- Back Right Trolley -->
+  <link name="back_right_wheel">
+    <collision><origin xyz="0 0 0" rpy="1.57 0 1.5708"/><geometry><sphere radius="0.0523"/></geometry></collision>
+    <inertial>
+      <origin xyz="0 0 0"/>
+      <mass value="0.1"/>
+      <inertia ixx="0.000144" iyy="0.000144" izz="0.000144"
+               ixy="0.0" ixz="0.0" iyz="0.0"/>
+    </inertial>
+  </link>
+  <joint name="back_right_wheel_joint" type="fixed">
+    <parent link="chassis_link"/>
+    <child link="back_right_wheel"/>
+    <origin xyz="-0.40 -0.27 -0.02" rpy="0 0 0"/>
+  </joint>
+  <!-- Middle Left Traction -->
+  <link name="middle_left_wheel">
+    <collision><origin xyz="0 0 0" rpy="1.57 0 1.5708"/>
+    <geometry><cylinder radius="0.0735" length="0.03"/></geometry></collision>
+        <!-- <visual>
       <origin xyz="0 0 0" rpy="0 0 0"/>
-      <mass value="24.5"/>
-      <inertia ixx="1.84514" ixy="0" ixz="0" iyy="1.04961" iyz="0" izz="1.04961"/>
-    </inertial>
-    <collision>
-      <origin xyz="0 0 0" rpy="0 1.5708 0"/>
-      <geometry><cylinder radius="0.072" length="0.06"/></geometry>
-    </collision>
-    <visual>
+      <geometry>
+        <mesh filename="package://alphabot_description/meshes/wheel.dae" scale="0.5 0.5 0.5"/>
+      </geometry>
+    </visual> -->
+    <inertial>
+      <origin xyz="0 0 0" rpy="-1.57 0 1.5708"/>
+      <mass value="1"/>
+      <inertia ixx="0.1" iyy="0.1" izz="0.1"
+               ixy="0.0" ixz="0.0" iyz="0.0"/>
+    </inertial>
+  </link>
+  <joint name="middle_left_wheel_joint" type="continuous">
+    <parent link="chassis_link"/>
+    <child link="middle_left_wheel"/>
+    <origin xyz="0 0.27 0" rpy="0 0 1.57"/>
+    <axis xyz="1 0 0"/>
+  </joint>
+  <!-- Middle Right Traction -->
+  <link name="middle_right_wheel">
+    <collision><origin xyz="0 0 0" rpy="1.57 0 1.5708"/><geometry><cylinder radius="0.0735" length="0.03"/></geometry></collision>
+        <!-- <visual>
       <origin xyz="0 0 0" rpy="0 0 0"/>
       <geometry>
         <mesh filename="package://alphabot_description/meshes/wheel.dae" scale="0.5 0.5 0.5"/>
       </geometry>
-    </visual>
-  </link>
-  <joint name="bl_axle" type="continuous">
-    <origin xyz="-0.18 -0.244 0" rpy="0 0 0"/>
-    <parent link="chassis_link"/>
-    <child  link="bl_1"/>
+    </visual> -->
+    <inertial>
+      <origin xyz="0 0 0" rpy="-1.57 0 1.5708"/>
+      <mass value="1"/>
+      <inertia ixx="0.1" iyy="0.1" izz="0.1"
+               ixy="0.0" ixz="0.0" iyz="0.0"/>
+    </inertial>
+  </link>
+  <joint name="middle_right_wheel_joint" type="continuous">
+    <parent link="chassis_link"/>
+    <child link="middle_right_wheel"/>
+    <origin xyz="0 -0.27 0" rpy="0 0 1.57"/>
     <axis xyz="1 0 0"/>
-    <dynamics friction="12.0316061502"/>
-  </joint>
-  <link name="br_1">
-    <inertial>
-      <origin xyz="0 0 0" rpy="0 0 0"/>
-      <mass value="24.5"/>
-      <inertia ixx="1.84514" ixy="0" ixz="0" iyy="1.04961" iyz="0" izz="1.04961"/>
-    </inertial>
-    <collision>
-      <origin xyz="0 0 0" rpy="0 1.5708 0"/>
-      <geometry><cylinder radius="0.072" length="0.06"/></geometry>
-    </collision>
-    <visual>
-      <origin xyz="0 0 0" rpy="0 0 0"/>
-      <geometry>
-        <mesh filename="package://alphabot_description/meshes/wheel.dae" scale="0.5 0.5 0.5"/>
-      </geometry>
-    </visual>
-  </link>
-  <joint name="br_axle" type="continuous">
-    <origin xyz="0.18 -0.244 0" rpy="0 0 0"/>
-    <parent link="chassis_link"/>
-    <child  link="br_1"/>
-    <axis xyz="1 0 0"/>
-    <dynamics friction="12.0316061502"/>
-  </joint>
-  <link name="l_steer_1">
-    <inertial><origin xyz="0 0 0"/><mass value="1"/><inertia ixx="1" ixy="0" ixz="0" iyy="1" iyz="0" izz="1"/></inertial>
-  </link>
-  <joint name="l_steer" type="revolute">
-    <origin xyz="-0.236 0.244 0" rpy="0 0 0"/>
-    <parent link="chassis_link"/>
-    <child  link="l_steer_1"/>
-    <axis xyz="0 0 1"/>
-    <limit lower="0.0" upper="0.0" effort="1e9" velocity="0.0"/>
-  </joint>
-  <link name="r_steer_1">
-    <inertial><origin xyz="0 0 0"/><mass value="1"/><inertia ixx="1" ixy="0" ixz="0" iyy="1" iyz="0" izz="1"/></inertial>
-  </link>
-  <joint name="r_steer" type="revolute">
-    <origin xyz="0.236 0.244 0" rpy="0 0 0"/>
-    <parent link="chassis_link"/>
-    <child  link="r_steer_1"/>
-    <axis xyz="0 0 1"/>
-    <limit lower="0.0" upper="0.0" effort="1e9" velocity="0.0"/>
-  </joint>
-  <link name="fl_1">
-    <inertial>
-      <origin xyz="0 0 0" rpy="0 0 0"/>
-      <mass value="24.5"/>
-      <inertia ixx="1.84514" ixy="0" ixz="0" iyy="1.04961" iyz="0" izz="1.04961"/>
-    </inertial>
-    <collision>
-      <origin xyz="0 0 0" rpy="0 1.5708 0"/>
-      <geometry><cylinder radius="0.072" length="0.06"/></geometry>
-    </collision>
-    <visual>
-      <origin xyz="0 0 0" rpy="0 0 0"/>
-      <geometry>
-        <mesh filename="package://alphabot_description/meshes/wheel.dae" scale="0.5 0.5 0.5"/>
-      </geometry>
-    </visual>
-  </link>
-  <joint name="fl_axle" type="continuous">
-    <origin xyz="0 0 0" rpy="0 0 0"/>
-    <parent link="l_steer_1"/>
-    <child  link="fl_1"/>
-    <axis xyz="1 0 0"/>
-  </joint>
-  <link name="fr_1">
-    <inertial>
-      <origin xyz="0 0 0" rpy="0 0 0"/>
-      <mass value="24.5"/>
-      <inertia ixx="1.84514" ixy="0" ixz="0" iyy="1.04961" iyz="0" izz="1.04961"/>
-    </inertial>
-    <collision>
-      <origin xyz="0 0 0" rpy="0 1.5708 0"/>
-      <geometry><cylinder radius="0.072" length="0.06"/></geometry>
-    </collision>
-    <visual>
-      <origin xyz="0 0 0" rpy="0 0 0"/>
-      <geometry>
-        <mesh filename="package://alphabot_description/meshes/wheel.dae" scale="0.5 0.5 0.5"/>
-      </geometry>
-    </visual>
-  </link>
-  <joint name="fr_axle" type="continuous">
-    <origin xyz="0 0 0" rpy="0 0 0"/>
-    <parent link="r_steer_1"/>
-    <child  link="fr_1"/>
-    <axis xyz="1 0 0"/>
-  </joint>
+  </joint>
+  <!-- ================= LIDAR ================= -->
   <link name="lidar_link">
-    <inertial><origin xyz="0 0 0"/><mass value="0.5"/><inertia ixx="0.001" ixy="0" ixz="0" iyy="0.001" iyz="0" izz="0.001"/></inertial>
-    <visual><origin xyz="0 0 0"/><geometry><cylinder radius="0.04" length="0.05"/></geometry></visual>
-    <collision><origin xyz="0 0 0"/><geometry><cylinder radius="0.04" length="0.05"/></geometry></collision>
+    <inertial>
+      <origin xyz="0 0 0"/>
+      <mass value="0.5"/>
+      <inertia ixx="0.001" iyy="0.001" izz="0.001"
+               ixy="0.0" ixz="0.0" iyz="0.0"/>
+    </inertial>
+    <visual><origin xyz="0 0 0"/><geometry><cylinder radius="0.02" length="0.03"/></geometry></visual>
+    <collision><origin xyz="0 0 0"/><geometry><cylinder radius="0.02" length="0.03"/></geometry></collision>
   </link>
   <joint name="lidar_joint" type="fixed">
-    <origin xyz="0 0 0.18" rpy="0 0 0"/>
+    <origin xyz="0 0 0.28" rpy="0 0 0"/>
     <parent link="link_base"/>
     <child  link="lidar_link"/>
   </joint>
-  <link name="lift_link">
-    <inertial><origin xyz="0 0 0"/><mass value="0.1"/><inertia ixx="0.001" ixy="0" ixz="0" iyy="0.001" iyz="0" izz="0.001"/></inertial>
-    <visual>
-      <origin xyz="0 0 0.1" rpy="0 0 0"/>
-      <geometry>
-        <mesh filename="package://alphabot_description/meshes/platform.dae" scale="0.5 0.5 0.5"/>
-      </geometry>
-    </visual>
-    <collision>
-      <origin xyz="0 0 0.1" rpy="0 0 0"/>
-      <geometry>
-      <mesh filename="package://alphabot_description/meshes/platform_collision.dae" scale="0.5 0.5 0.5"/>
-      </geometry>
-    </collision>
-  </link>
-  <joint name="lift_fixed_joint" type="fixed">
-    <origin xyz="0 0 0.02" rpy="0 0 0"/>
-    <parent link="lidar_link"/>
-    <child  link="lift_link"/>
-  </joint>
   <link name="realsense_link">
     <inertial>
-      <origin xyz="0 0 0" rpy="0 0 1.57"/>
+      <origin xyz="0 0 0" rpy="1.57 1.57 1.57"/>
       <mass value="0.0615752"/>
       <inertia ixx="9.108e-05" ixy="0" ixz="0" iyy="2.51e-06" iyz="0" izz="8.931e-05"/>
@@ -241,18 +219,20 @@
   </gazebo>
   <gazebo reference="chassis_link"><selfCollide>true</selfCollide><mu1>0.2</mu1><mu2>0.2</mu2></gazebo>
-  <gazebo reference="bl_1"><mu1>1e6</mu1><mu2>1e6</mu2></gazebo>
-  <gazebo reference="br_1"><mu1>1e6</mu1><mu2>1e6</mu2></gazebo>
-  <gazebo reference="fl_1"><mu1>1e6</mu1><mu2>1e6</mu2></gazebo>
-  <gazebo reference="fr_1"><mu1>1e6</mu1><mu2>1e6</mu2></gazebo>
+  <gazebo reference="front_left_wheel"><mu1>1e6</mu1><mu2>1e6</mu2></gazebo>
+  <gazebo reference="front_right_wheel"><mu1>1e6</mu1><mu2>1e6</mu2></gazebo>
+  <gazebo reference="back_left_wheel"><mu1>1e6</mu1><mu2>1e6</mu2></gazebo>
+  <gazebo reference="back_right_wheel"><mu1>1e6</mu1><mu2>1e6</mu2></gazebo>
+  <gazebo reference="middle_left_wheel"><mu1>1e6</mu1><mu2>1e6</mu2></gazebo>
+  <gazebo reference="middle_right_wheel"><mu1>1e6</mu1><mu2>1e6</mu2></gazebo>
   <gazebo reference="lift_link"><mu1>1e6</mu1><mu2>1e5</mu2><kp>1e5</kp><kd>1</kd><maxVel>0.01</maxVel><minDepth>0.001</minDepth></gazebo>
   <gazebo reference="lidar_link">
     <sensor name="amr_lidar" type="ray">
       <always_on>true</always_on>
-      <update_rate>15</update_rate> <!-- 10-15 Hz like real sensors -->
+      <update_rate>15</update_rate>
       <visualize>true</visualize>
       <ray>
         <scan>
           <horizontal>
-            <samples>1080</samples>        <!-- 0.33° per beam -->
+            <samples>1080</samples>
             <resolution>1</resolution>
             <min_angle>-3.14159265</min_angle>
@@ -281,27 +261,25 @@
     </sensor>
   </gazebo>
+  <!-- ================= JOINT STATE PUBLISHER ================= -->
   <gazebo>
     <plugin name="joint_state_publisher" filename="libgazebo_ros_joint_state_publisher.so">
       <update_rate>100</update_rate>
-      <joint_name>bl_axle</joint_name>
-      <joint_name>br_axle</joint_name>
-      <joint_name>fl_axle</joint_name>
-      <joint_name>fr_axle</joint_name>
-      <joint_name>l_steer</joint_name>
-      <joint_name>r_steer</joint_name>
+      <joint_name>middle_left_wheel_joint</joint_name>
+      <joint_name>middle_right_wheel_joint</joint_name>
     </plugin>
   </gazebo>
+  <!-- ================= DIFF DRIVE ================= -->
   <gazebo>
     <plugin name="diff_drive" filename="libgazebo_ros_diff_drive.so">
       <ros>
-      <parameter name="use_sim_time" value="true"/>
-      <remapping>cmd_vel:=/cmd_vel</remapping>
-      <remapping>odom:=/odom</remapping>
+        <parameter name="use_sim_time" value="true"/>
+        <remapping>cmd_vel:=/cmd_vel</remapping>
+        <remapping>odom:=/odom</remapping>
       </ros>
       <update_rate>100</update_rate>
-      <left_joint>bl_axle</left_joint>
-      <right_joint>br_axle</right_joint>
-      <wheel_diameter>0.144</wheel_diameter>
-      <wheel_separation>0.488</wheel_separation>
+      <left_joint>middle_left_wheel_joint</left_joint>
+      <right_joint>middle_right_wheel_joint</right_joint>
+      <wheel_diameter>0.146</wheel_diameter>
+      <wheel_separation>0.54</wheel_separation>
       <max_wheel_torque>1000</max_wheel_torque>
       <max_wheel_acceleration>0.0</max_wheel_acceleration>
