Commit message: Added new urdf

File: ALPHA_BOT/alphabot_description/urdf/alphabot.urdf.xacro (robot description, xacro)
@@ -1,294 +1,165 @@
 <?xml version="1.0"?>
-<robot name="alphabot" xmlns:xacro="http://www.ros.org/wiki/xacro">
-  <xacro:arg name="scan_topic" default="/scan"/>
-  <xacro:arg name="cmd_vel_topic" default="/amazon_robot/cmd_vel"/>
-  <xacro:arg name="odom_topic" default="/amazon_robot/odom"/>
-  <xacro:arg name="use_gazebo_camera" default="true"/>
-  <link name="base_footprint"/>
-  <link name="link_base"/>
-  <joint name="base_joint" type="fixed">
-    <parent link="base_footprint"/>
-    <child  link="link_base"/>
-    <origin xyz="0 0 0.072" rpy="0 0 0"/>
-  </joint>
-  <link name="chassis_link">
-    <inertial>
-      <origin xyz="0 0 0" rpy="0 0 1.57"/>
-      <mass value="1580"/>
-      <inertia ixx="1997.86" ixy="0" ixz="0" iyy="442.769" iyz="62.5206" izz="2238.05"/>
-    </inertial>
-    <visual>
-      <origin xyz="0 0 0" rpy="0 0 1.57"/>
-      <geometry>
-        <mesh filename="package://alphabot_description/meshes/chassy.dae" scale="1 1 1"/>
-      </geometry>
-    </visual>
-    <collision>
-      <origin xyz="0 0 0" rpy="0 0 1.57"/>
-      <geometry>
-        <mesh filename="package://alphabot_description/meshes/chassy.dae" scale="1 1 1"/>
-      </geometry>
-    </collision>
-  </link>
-  <joint name="chassis_link_joint" type="fixed">
-    <parent link="link_base"/>
-    <child  link="chassis_link"/>
-    <origin xyz="0 0 0" rpy="0 0 0"/>
-  </joint>
-  <!-- ================= WHEELS (6 TOTAL, rotated Z) ================= -->
-  <!-- Front Left Trolley -->
-  <link name="front_left_wheel">
-    <collision><origin xyz="0 0 0" rpy="1.57 0 1.5708"/><geometry><sphere radius="0.0523"/></geometry></collision>
-    <inertial>
-      <origin xyz="0 0 0"/>
-      <mass value="0.1"/>
-      <inertia ixx="0.000144" iyy="0.000144" izz="0.000144"
-               ixy="0.0" ixz="0.0" iyz="0.0"/>
-    </inertial>
-  </link>
-  <joint name="front_left_wheel_joint" type="fixed">
-    <parent link="chassis_link"/>
-    <child link="front_left_wheel"/>
-    <origin xyz="0.40 0.27 -0.02" rpy="0 0 0"/>
-  </joint>
-  <!-- Front Right Trolley -->
-  <link name="front_right_wheel">
-    <collision><origin xyz="0 0 0" rpy="1.57 0 1.5708"/><geometry><sphere radius="0.0523"/></geometry></collision>
-    <inertial>
-      <origin xyz="0 0 0"/>
-      <mass value="0.1"/>
-      <inertia ixx="0.000144" iyy="0.000144" izz="0.000144"
-               ixy="0.0" ixz="0.0" iyz="0.0"/>
-    </inertial>
-  </link>
-  <joint name="front_right_wheel_joint" type="fixed">
-    <parent link="chassis_link"/>
-    <child link="front_right_wheel"/>
-    <origin xyz="0.40 -0.27 -0.02" rpy="0 0 0"/>
-  </joint>
-  <!-- Back Left Trolley -->
-  <link name="back_left_wheel">
-    <collision><origin xyz="0 0 0" rpy="1.57 0 1.5708"/><geometry><sphere radius="0.0523"/></geometry></collision>
-    <inertial>
-      <origin xyz="0 0 0"/>
-      <mass value="0.1"/>
-      <inertia ixx="0.000144" iyy="0.000144" izz="0.000144"
-               ixy="0.0" ixz="0.0" iyz="0.0"/>
-    </inertial>
-  </link>
-  <joint name="back_left_wheel_joint" type="fixed">
-    <parent link="chassis_link"/>
-    <child link="back_left_wheel"/>
-    <origin xyz="-0.40 0.27 -0.02" rpy="0 0 0"/>
-  </joint>
-  <!-- Back Right Trolley -->
-  <link name="back_right_wheel">
-    <collision><origin xyz="0 0 0" rpy="1.57 0 1.5708"/><geometry><sphere radius="0.0523"/></geometry></collision>
-    <inertial>
-      <origin xyz="0 0 0"/>
-      <mass value="0.1"/>
-      <inertia ixx="0.000144" iyy="0.000144" izz="0.000144"
-               ixy="0.0" ixz="0.0" iyz="0.0"/>
-    </inertial>
-  </link>
-  <joint name="back_right_wheel_joint" type="fixed">
-    <parent link="chassis_link"/>
-    <child link="back_right_wheel"/>
-    <origin xyz="-0.40 -0.27 -0.02" rpy="0 0 0"/>
-  </joint>
-  <!-- Middle Left Traction -->
-  <link name="middle_left_wheel">
-    <collision><origin xyz="0 0 0" rpy="1.57 0 1.5708"/>
-    <geometry><cylinder radius="0.0735" length="0.03"/></geometry></collision>
-        <!-- <visual>
-      <origin xyz="0 0 0" rpy="0 0 0"/>
-      <geometry>
-        <mesh filename="package://alphabot_description/meshes/wheel.dae" scale="0.5 0.5 0.5"/>
-      </geometry>
-    </visual> -->
-    <inertial>
-      <origin xyz="0 0 0" rpy="-1.57 0 1.5708"/>
-      <mass value="1"/>
-      <inertia ixx="0.1" iyy="0.1" izz="0.1"
-               ixy="0.0" ixz="0.0" iyz="0.0"/>
-    </inertial>
-  </link>
-  <joint name="middle_left_wheel_joint" type="continuous">
-    <parent link="chassis_link"/>
-    <child link="middle_left_wheel"/>
-    <origin xyz="0 0.27 0" rpy="0 0 1.57"/>
-    <axis xyz="1 0 0"/>
-  </joint>
-  <!-- Middle Right Traction -->
-  <link name="middle_right_wheel">
-    <collision><origin xyz="0 0 0" rpy="1.57 0 1.5708"/><geometry><cylinder radius="0.0735" length="0.03"/></geometry></collision>
-        <!-- <visual>
-      <origin xyz="0 0 0" rpy="0 0 0"/>
-      <geometry>
-        <mesh filename="package://alphabot_description/meshes/wheel.dae" scale="0.5 0.5 0.5"/>
-      </geometry>
-    </visual> -->
-    <inertial>
-      <origin xyz="0 0 0" rpy="-1.57 0 1.5708"/>
-      <mass value="1"/>
-      <inertia ixx="0.1" iyy="0.1" izz="0.1"
-               ixy="0.0" ixz="0.0" iyz="0.0"/>
-    </inertial>
-  </link>
-  <joint name="middle_right_wheel_joint" type="continuous">
-    <parent link="chassis_link"/>
-    <child link="middle_right_wheel"/>
-    <origin xyz="0 -0.27 0" rpy="0 0 1.57"/>
-    <axis xyz="1 0 0"/>
-  </joint>
-  <!-- ================= LIDAR ================= -->
-  <link name="lidar_link">
-    <inertial>
-      <origin xyz="0 0 0"/>
-      <mass value="0.5"/>
-      <inertia ixx="0.001" iyy="0.001" izz="0.001"
-               ixy="0.0" ixz="0.0" iyz="0.0"/>
-    </inertial>
-    <visual><origin xyz="0 0 0"/><geometry><cylinder radius="0.02" length="0.03"/></geometry></visual>
-    <collision><origin xyz="0 0 0"/><geometry><cylinder radius="0.02" length="0.03"/></geometry></collision>
-  </link>
-  <joint name="lidar_joint" type="fixed">
-    <origin xyz="0 0 0.28" rpy="0 0 0"/>
-    <parent link="link_base"/>
-    <child  link="lidar_link"/>
-  </joint>
-  <link name="realsense_link">
-    <inertial>
-      <origin xyz="0 0 0" rpy="1.57 1.57 1.57"/>
-      <mass value="0.0615752"/>
-      <inertia ixx="9.108e-05" ixy="0" ixz="0" iyy="2.51e-06" iyz="0" izz="8.931e-05"/>
-    </inertial>
-    <visual name="visual">
-      <origin xyz="0 0 0" rpy="0 0 1.57"/>
-      <geometry>
-        <mesh filename="package://alphabot_description/meshes/RealSense_D435/meshes/realsense.dae"/>
-      </geometry>
-    </visual>
-    <collision name="collision">
-     <origin xyz="0 0 0" rpy="0 0 1.57"/>
-      <geometry>
-        <mesh filename="package://alphabot_description/meshes/RealSense_D435/meshes/realsense.dae"/>
-      </geometry>
-    </collision>
-  </link>
-  <joint name="realsense_joint" type="fixed">
-    <origin xyz="0 0.45 0.15" rpy="0 0 1.57"/>
-    <parent link="link_base"/>
-    <child  link="realsense_link"/>
-  </joint>
-  <link name="realsense_depth_frame"/>
-  <joint name="realsense_depth_frame_joint" type="fixed">
-    <origin xyz="0 0 0" rpy="-1.57 0 3.14"/>
-    <parent link="realsense_link"/>
-    <child  link="realsense_depth_frame"/>
-  </joint>
-  <link name="realsense_depth_optical_frame"/>
-  <joint name="realsense_depth_optical_joint" type="fixed">
-    <origin xyz="0 0 0" rpy="-1.57 -1.57 1.57"/>
-    <parent link="realsense_depth_frame"/>
-    <child  link="realsense_depth_optical_frame"/>
-  </joint>
-  <gazebo reference="realsense_link">
-    <sensor name="realsense_depth_camera" type="depth">
-      <always_on>1</always_on>
-      <update_rate>30</update_rate>
-      <visualize>0</visualize>
-      <pose>0 0 0 0 0 0</pose>
-      <camera name="depth_camera">
-        <horizontal_fov>1.0472</horizontal_fov>
-        <image><width>640</width><height>480</height><format>B8G8R8</format></image>
-        <clip><near>0.01</near><far>10</far></clip>
-      </camera>
-      <plugin name="realsense_depth_plugin" filename="libgazebo_ros_camera.so">
-        <ros>
-          <remapping>image_raw:=/realsense_depth_camera/depth/image_raw</remapping>
-          <remapping>camera_info:=/realsense_depth_camera/depth/camera_info</remapping>
-          <remapping>points:=/realsense_depth_camera/points</remapping>
-        </ros>
-        <frame_name>realsense_depth_optical_frame</frame_name>
-        <output_pointcloud>true</output_pointcloud>
-        <pointCloudCutoff>0.01</pointCloudCutoff>
-        <pointCloudCutoffMax>10.0</pointCloudCutoffMax>
-      </plugin>
-    </sensor>
-  </gazebo>
-  <gazebo reference="chassis_link"><selfCollide>true</selfCollide><mu1>0.2</mu1><mu2>0.2</mu2></gazebo>
-  <gazebo reference="front_left_wheel"><mu1>1e6</mu1><mu2>1e6</mu2></gazebo>
-  <gazebo reference="front_right_wheel"><mu1>1e6</mu1><mu2>1e6</mu2></gazebo>
-  <gazebo reference="back_left_wheel"><mu1>1e6</mu1><mu2>1e6</mu2></gazebo>
-  <gazebo reference="back_right_wheel"><mu1>1e6</mu1><mu2>1e6</mu2></gazebo>
-  <gazebo reference="middle_left_wheel"><mu1>1e6</mu1><mu2>1e6</mu2></gazebo>
-  <gazebo reference="middle_right_wheel"><mu1>1e6</mu1><mu2>1e6</mu2></gazebo>
-  <gazebo reference="lift_link"><mu1>1e6</mu1><mu2>1e5</mu2><kp>1e5</kp><kd>1</kd><maxVel>0.01</maxVel><minDepth>0.001</minDepth></gazebo>
-  <gazebo reference="lidar_link">
-    <sensor name="amr_lidar" type="ray">
-      <always_on>true</always_on>
-      <update_rate>15</update_rate>
-      <visualize>true</visualize>
-      <ray>
-        <scan>
-          <horizontal>
-            <samples>1080</samples>
-            <resolution>1</resolution>
-            <min_angle>-3.14159265</min_angle>
-            <max_angle>3.14159265</max_angle>
-          </horizontal>
-        </scan>
-        <range>
-          <min>0.12</min>       <!-- avoid robot self-collision -->
-          <max>25.0</max>       <!-- typical outdoor lidar range -->
-          <resolution>0.001</resolution>
-        </range>
-        <noise>
-          <type>gaussian</type>
-          <mean>0.0</mean>
-          <stddev>0.01</stddev>  <!-- 1 cm noise, realistic -->
-        </noise>
-      </ray>
-      <plugin name="gazebo_ros_ray_sensor" filename="libgazebo_ros_ray_sensor.so">
-        <ros>
-          <parameter name="use_sim_time" value="true"/>
-          <remapping>~/out:=/scan</remapping> <!-- topic published -->
-        </ros>
-        <output_type>sensor_msgs/LaserScan</output_type>
-        <frame_name>lidar_link</frame_name>
-      </plugin>
-    </sensor>
-  </gazebo>
-  <!-- ================= JOINT STATE PUBLISHER ================= -->
-  <gazebo>
-    <plugin name="joint_state_publisher" filename="libgazebo_ros_joint_state_publisher.so">
-      <update_rate>100</update_rate>
-      <joint_name>middle_left_wheel_joint</joint_name>
-      <joint_name>middle_right_wheel_joint</joint_name>
-    </plugin>
-  </gazebo>
-  <!-- ================= DIFF DRIVE ================= -->
-  <gazebo>
-    <plugin name="diff_drive" filename="libgazebo_ros_diff_drive.so">
-      <ros>
-        <parameter name="use_sim_time" value="true"/>
-        <remapping>cmd_vel:=/cmd_vel</remapping>
-        <remapping>odom:=/odom</remapping>
-      </ros>
-      <update_rate>100</update_rate>
-      <left_joint>middle_left_wheel_joint</left_joint>
-      <right_joint>middle_right_wheel_joint</right_joint>
-      <wheel_diameter>0.146</wheel_diameter>
-      <wheel_separation>0.54</wheel_separation>
-      <max_wheel_torque>1000</max_wheel_torque>
-      <max_wheel_acceleration>0.0</max_wheel_acceleration>
-      <publish_odom>true</publish_odom>
-      <publish_odom_tf>true</publish_odom_tf>
-      <publish_wheel_tf>true</publish_wheel_tf>
-      <odometry_frame>odom</odometry_frame>
-      <robot_base_frame>base_footprint</robot_base_frame>
-      <odometry_source>0</odometry_source>
-    </plugin>
-  </gazebo>
+<robot xmlns:xacro="http://www.ros.org/wiki/xacro" name="bcr_bot">
+    <xacro:property name="chassis_mass" value="70"/>
+    <xacro:property name="chassis_length" value="0.9"/>
+    <xacro:property name="chassis_width" value="0.64"/>
+    <xacro:property name="chassis_height" value="0.19"/>
+    <xacro:property name="traction_wheel_mass" value="1"/>
+    <xacro:property name="traction_wheel_base" value="0.88"/>
+    <xacro:property name="traction_max_wheel_torque" value="20000"/>
+    <xacro:property name="traction_wheel_friction" value="5.0"/>
+    <xacro:property name="trolley_wheel_mass" value="0.1"/>
+    <xacro:property name="trolley_track_width" value="0.54"/>
+    <xacro:property name="trolley_wheel_friction" value="0.0"/>
+    <xacro:property name="trolley_wheel_radius" value="0.06"/>
+    <xacro:property name="eps" value="0.002"/>
+    <xacro:property name="traction_wheel_radius" value="0.1"/>
+    <xacro:property name="traction_wheel_width" value="0.05"/>
+    <xacro:property name="traction_track_width" value="0.6"/>
+    <xacro:property name="two_d_lidar_update_rate" value="30"/>
+    <xacro:property name="two_d_lidar_sample_size" value="361"/>
+    <xacro:property name="two_d_lidar_min_angle" value="0"/>
+    <xacro:property name="two_d_lidar_max_angle" value="360"/>
+    <xacro:property name="two_d_lidar_min_range" value="0.55"/>
+    <xacro:property name="two_d_lidar_max_range" value="16"/>
+    <xacro:property name="camera_baseline" value="0.06"/>
+    <xacro:property name="camera_height" value="0.10"/>
+    <xacro:property name="camera_horizontal_fov" value="60"/>
+    <xacro:arg name="robot_namespace" default=""/>
+    <xacro:arg name="wheel_odom_topic" default="odom" />
+    <xacro:arg name="camera_enabled" default="true" />
+    <xacro:arg name="stereo_camera_enabled" default="false" />
+    <xacro:arg name="two_d_lidar_enabled" default="true" />
+    <xacro:arg name="publish_wheel_odom_tf" default="true" />
+    <xacro:arg name="conveyor_enabled" default="false"/>
+    <xacro:arg name="ground_truth_frame" default="map"/>
+    <xacro:arg name="sim_gazebo" default="true" />
+    <xacro:arg name="sim_ign" default="false" />
+    <xacro:arg name="sim_gz" default="false" />
+    <xacro:arg name="odometry_source" default="world" />
+    <xacro:property name="odometry_source" value="$(arg odometry_source)"/>
+    <xacro:include filename="$(find alphabot_description)/urdf/materials.xacro"/>
+    <xacro:include filename="$(find alphabot_description)/urdf/macros.xacro"/>
+    <xacro:include filename="$(find alphabot_description)/urdf/gazebo.xacro"/>
+    <link name="base_footprint"/>
+    <link name="link_base"/>
+    <joint name="base_joint" type="fixed">
+        <parent link="base_footprint"/>
+        <child link="link_base"/>
+        <origin xyz="0.0 0 ${chassis_height/2 + traction_wheel_radius}" rpy="0 0 0.0" />
+    </joint>
+    <link name="chassis_link">
+        <collision>
+            <origin xyz="0 0 -0.05" rpy="0 0 0" />
+            <geometry>
+                <box size="${chassis_length} ${chassis_width} ${chassis_height}"/>
+            </geometry>
+        </collision>
+        <visual>
+            <origin xyz="0 0 -0.205" rpy="0 0 0" />
+            <geometry>
+                <mesh filename="file://$(find alphabot_description)/meshes/chassy.dae" scale="1 1 1"/>
+            </geometry>
+        </visual>
+        <inertial>
+            <mass value="${chassis_mass}" />
+            <xacro:box_inertia m="${chassis_mass}" x="${chassis_length}" y="${chassis_width}" z = "${chassis_height}"/>
+        </inertial>
+    </link>
+    <joint name="chassis_joint" type="fixed">
+        <parent link="link_base"/>
+        <child link="chassis_link"/>
+        <origin xyz="0.0 0 0" rpy="0 0 0.0" />
+    </joint>
+    <xacro:trolley_wheel cardinality="front" dexterity="left" origin_x="${chassis_length/2}" origin_y="${trolley_track_width/2}" origin_z="-${trolley_wheel_radius+chassis_height/2}"/>
+    <xacro:trolley_wheel cardinality="front" dexterity="right" origin_x="${chassis_length/2}" origin_y="-${trolley_track_width/2}" origin_z="-${trolley_wheel_radius+chassis_height/2}"/>
+    <xacro:trolley_wheel cardinality="back" dexterity="left" origin_x="-${chassis_length/2}" origin_y="${trolley_track_width/2}" origin_z="-${trolley_wheel_radius+chassis_height/2}"/>
+    <xacro:trolley_wheel cardinality="back" dexterity="right" origin_x="-${chassis_length/2}" origin_y="-${trolley_track_width/2}" origin_z="-${trolley_wheel_radius+chassis_height/2}"/>
+    <xacro:traction_wheel cardinality="middle" dexterity="left" origin_x="0" origin_y="${traction_track_width/2}" origin_z="-${chassis_height/2+2*trolley_wheel_radius+eps-traction_wheel_radius}"/>
+    <xacro:traction_wheel cardinality="middle" dexterity="right" origin_x="0" origin_y="-${traction_track_width/2}" origin_z="-${chassis_height/2+2*trolley_wheel_radius+eps-traction_wheel_radius}"/>
+    <xacro:if value="$(arg two_d_lidar_enabled)">
+        <link name="two_d_lidar">
+            <collision>
+                <origin xyz="0 0 0" rpy="0 0 0" />
+                <geometry>
+                    <cylinder length="0.06" radius="0.075"/>
+                </geometry>
+            </collision>
+            <visual>
+                <origin xyz="0 0 0" rpy="0 0 0" />
+                <geometry>
+                    <cylinder length="0.06" radius="0.075"/>
+                </geometry>
+                <material name="aluminium"/>
+            </visual>
+            <inertial>
+                <origin xyz="0 0 0" rpy="0 0 0" />
+                <mass value="0.1"/>
+                <xacro:cylinder_inertia m="0.1" r="0.075" h="0.06"/>
+            </inertial>
+        </link>
+        <joint name="two_d_lidar_joint" type="fixed">
+            <parent link="link_base"/>
+            <child link="two_d_lidar"/>
+            <origin xyz="0.0 0 0.08" rpy="0 0 0" />
+        </joint>
+        <gazebo reference="two_d_lidar">
+            <material>Gazebo/White</material>
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
File: MOBILE_MANIPULATOR/mobile_manipulator_description/urdf/mobile_manipulator.urdf.xacro (robot description, xacro)
@@ -15,10 +15,4 @@
     <origin xyz="0 -0.25 0.06" rpy="0 0 0"/>
   </joint>
-<!--
-  <link name="world"/>
-  <joint name="world_to_robot" type="fixed">
-    <parent link="world"/>
-    <child link="base_footprint"/>
-  </joint> -->
   <gazebo>
     <plugin filename="libgazebo_ros2_control.so" name="gazebo_ros2_control">

File: MOBILE_MANIPULATOR/mobile_manipulator_description/urdf/mobile_manipulator_ros_contol.xacro (robot description, xacro)
@@ -1,10 +1,8 @@
 <?xml version="1.0"?>
 <robot name="mobile_manipulator" xmlns:xacro="http://www.ros.org/wiki/xacro">
-  <!-- ros2_control setup -->
   <ros2_control name="GazeboSystem" type="system">
     <hardware>
       <plugin>gazebo_ros2_control/GazeboSystem</plugin>
     </hardware>
-    <!-- Slider -->
     <joint name="slider_joint">
       <command_interface name="position"/>
@@ -12,5 +10,4 @@
       <state_interface name="velocity"/>
     </joint>
-    <!-- 7 DOF Arm -->
     <joint name="joint1">
       <command_interface name="position"/>
@@ -49,5 +46,4 @@
     </joint>
   </ros2_control>
-  <!-- Transmissions for each controllable joint -->
   <transmission name="slider_trans">
     <type>transmission_interface/SimpleTransmission</type>

Commit message: Solved the plugin issue and corrected teh linear guide pose

File: ALPHA_BOT/alphabot_description/urdf/alphabot.urdf.xacro (robot description, xacro)
@@ -21,5 +21,5 @@
     <xacro:property name="two_d_lidar_min_angle" value="0"/>
     <xacro:property name="two_d_lidar_max_angle" value="360"/>
-    <xacro:property name="two_d_lidar_min_range" value="0.55"/>
+    <xacro:property name="two_d_lidar_min_range" value="0.12"/>
     <xacro:property name="two_d_lidar_max_range" value="16"/>
     <xacro:property name="camera_baseline" value="0.06"/>

File: ALPHA_BOT/alphabot_description/urdf/gazebo.xacro (robot description, xacro)
@@ -56,7 +56,7 @@
         <gazebo reference="two_d_lidar">
             <gravity>true</gravity>
-            <sensor type="ray" name="two_d_lidar">
+            <sensor type="gpu_ray" name="two_d_lidar">
                 <pose>0 0 0 0 0 0</pose>
-                <visualize>false</visualize>
+                <visualize>true</visualize>
                 <update_rate>${two_d_lidar_update_rate}</update_rate>
                 <ray>
@@ -82,5 +82,5 @@
                 <plugin name="gazebo_ros_laser" filename="libgazebo_ros_ray_sensor.so">
                     <ros>
-                        <remapping>~/out:=$(arg robot_namespace)/scan</remapping>
+                        <remapping>~/out:=scan</remapping>
                     </ros>
                     <output_type>sensor_msgs/LaserScan</output_type>

File: MOBILE_MANIPULATOR/mobile_manipulator_description/urdf/linear_guide.xacro (robot description, xacro)
@@ -6,5 +6,5 @@
         <box size="0.08 0.08 0.8"/>
       </geometry>
-      <origin xyz="0 -0.1 0.37" rpy="0 0 0"/>
+      <origin xyz="0 -0.1 0.42" rpy="0 0 0"/>
       <material name="grey">
         <color rgba="0.5 0.5 0.5 0.8"/>

File: MOBILE_MANIPULATOR/mobile_manipulator_description/urdf/mobile_manipulator.urdf.xacro (robot description, xacro)
@@ -8,10 +8,10 @@
     <parent link="chassis_link"/>
     <child  link="column"/>
-    <origin xyz="0 0 0.33" rpy="0 0 0"/>
+    <origin xyz="0 0 0.1" rpy="0 0 1.57"/>
   </joint>
   <joint name="slider_to_arm_base" type="fixed">
     <parent link="slider"/>
     <child  link="base_link"/>
-    <origin xyz="0 -0.25 0.06" rpy="0 0 0"/>
+    <origin xyz="0 -0.33 0.06" rpy="0 0 0"/>
   </joint>
   <gazebo>

Commit message: Added bt tree and elevator checking plugin

File: ALPHA_BOT/alphabot_description/urdf/alphabot.urdf.xacro (robot description, xacro)
@@ -47,5 +47,5 @@
         <parent link="base_footprint"/>
         <child link="link_base"/>
-        <origin xyz="0.0 0 ${chassis_height/2 + traction_wheel_radius}" rpy="0 0 0.0" />
+        <origin xyz="0 0.0 ${chassis_height/2 + traction_wheel_radius}" rpy="0 0 1.57" />
     </joint>
     <link name="chassis_link">

File: MOBILE_MANIPULATOR/mobile_manipulator_description/urdf/mobile_manipulator.urdf.xacro (robot description, xacro)
@@ -23,12 +23,10 @@
   </gazebo>
       <gazebo>
-        <plugin name="elevator_trigger_plugin" filename="libelevator_trigger_plugin.so">
-        <!-- Elevator entry position -->
+        <plugin name="amr_elevator_trigger_plugin" filename="libamr_elevator_trigger_plugin.so">
         <target_pose_enter>
-            <x>2.0</x>
-            <y>1.5</y>
-            <z>0.0</z>
+            <x>-3.498</x>
+            <y>0.017</y>
+            <z>0.534</z>
         </target_pose_enter>
-        <!-- Elevator exit position -->
         <target_pose_exit>
             <x>5.0</x>
@@ -36,5 +34,4 @@
             <z>0.0</z>
         </target_pose_exit>
-        <!-- Distance tolerance in meters -->
         <tolerance>0.5</tolerance>
         </plugin>
