Commit message: Added camere on robot

File: ALPHA_BOT/alphabot_description/urdf/alphabot.urdf.xacro (robot description, xacro)
@@ -47,5 +47,5 @@
         <parent link="base_footprint"/>
         <child link="link_base"/>
-        <origin xyz="0 0.0 ${chassis_height/2 + traction_wheel_radius}" rpy="0 0 1.57" />
+        <origin xyz="-0.6 17.8 ${chassis_height/2 + traction_wheel_radius}" rpy="0 0 1.57" />
     </joint>
     <link name="chassis_link">

File: MOBILE_MANIPULATOR/mobile_manipulator_description/urdf/camera_module.urdf.xacro (robot description, xacro)
@@ -1,51 +1,44 @@
 <?xml version="1.0"?>
 <robot xmlns:xacro="http://ros.org/wiki/xacro">
-  <!-- Macro for Intel Realsense D435 Camera -->
   <xacro:macro name="intel_d435_camera">
-    <!-- Camera main link -->
-    <link name="camera_link">
+    <link name="camera_link_base">
       <visual>
-        <origin xyz="0 0 0" rpy="1.57 0 1.57"/>
+        <origin xyz="0 0 0" rpy="0 0 1.57"/>
         <geometry>
-          <!-- <box size="0.3 0.3 0.05"/>  -->
-          <mesh filename="$(find mobile_manipulator_description)/meshes/kkk.stl" scale="1 1 1"/>
+          <mesh filename="$(find mobile_manipulator_description)/meshes/realsense.dae" scale="1 1 1"/>
         </geometry>
         <material name="Grey">
-          <color rgba="0.3 0.3 0.3 1.0"/>
+          <color rgba="0.8 0.8 0.8 1.0"/>
         </material>
       </visual>
       <collision>
-        <origin xyz="0 0 0" rpy="0 0 0"/>
+        <origin xyz="0 0 0" rpy="0 0 1.57"/>
         <geometry>
-          <!-- <box size="0.3 0.3 0.05"/>  -->
-          <mesh filename="$(find mobile_manipulator_description)/meshes/kkk.stl" scale="1 1 1"/>
+          <mesh filename="$(find mobile_manipulator_description)/meshes/realsense.dae" scale="1 1 1"/>
         </geometry>
       </collision>
       <inertial>
-        <origin xyz="0 0 0" rpy="0 0 0"/>
-        <mass value="0.05"/>
-        <inertia ixx="1e-3" ixy="0" ixz="0" iyy="1e-3" iyz="0" izz="1e-3"/>
+        <origin xyz="0 0 0" rpy="1.57 0 1.57"/>
+        <mass value="0.0615752"/>
+        <inertia ixx="9.108e-05" ixy="0" ixz="0" iyy="2.51e-06" iyz="0" izz="8.931e-05"/>
       </inertial>
     </link>
-    <!-- RGB Optical Frame -->
+    <link name="camera_rgb_link"/>
+    <joint name="camera_rgb_joint" type="fixed">
+      <parent link="camera_link_base"/>
+      <child link="camera_rgb_link"/>
+      <origin xyz="0 0 0" rpy="0 0 0"/>
+    </joint>
     <link name="camera_rgb_optical_frame"/>
     <joint name="camera_rgb_optical_joint" type="fixed">
-      <parent link="camera_link"/>
+      <parent link="camera_rgb_link"/>
       <child link="camera_rgb_optical_frame"/>
       <origin xyz="0 0 0" rpy="-1.5708 0 -1.5708"/>
     </joint>
-    <!-- Depth Optical Frame -->
-    <link name="camera_depth_optical_frame"/>
-    <joint name="camera_depth_optical_joint" type="fixed">
-      <parent link="camera_link"/>
-      <child link="camera_depth_optical_frame"/>
-      <origin xyz="0 0 0" rpy="-1.5708 0 -1.5708"/>
-    </joint>
-    <!-- Gazebo plugin for RGB camera -->
-    <gazebo reference="camera_link">
+    <gazebo reference="camera_rgb_link">
       <sensor name="d435_rgb" type="camera">
         <update_rate>30.0</update_rate>
         <camera>
-          <horizontal_fov>1.39626</horizontal_fov>
+          <horizontal_fov>1.0472</horizontal_fov>
           <image>
             <width>640</width>
@@ -54,13 +47,13 @@
           </image>
           <clip>
-            <near>0.1</near>
+            <near>0.01</near>
             <far>10.0</far>
           </clip>
         </camera>
-        <plugin name="d435_rgb_plugin" filename="libgazebo_ros_camera.so">
+        <plugin name="rgb_camera_controller" filename="libgazebo_ros_camera.so">
           <ros>
-            <namespace>/d435/rgb</namespace>
+            <namespace>/camera_rgb</namespace>
           </ros>
-          <camera_name>rgb</camera_name>
+          <camera_name>rgb_camera</camera_name>
           <image_topic_name>image_raw</image_topic_name>
           <camera_info_topic_name>camera_info</camera_info_topic_name>
@@ -69,32 +62,45 @@
       </sensor>
     </gazebo>
-    <!-- Gazebo plugin for Depth camera -->
-    <gazebo reference="camera_link">
+    <link name="camera_depth_link"/>
+    <joint name="camera_depth_joint" type="fixed">
+      <parent link="camera_link_base"/>
+      <child link="camera_depth_link"/>
+      <origin xyz="0 0 0" rpy="0 0 0"/>
+    </joint>
+    <link name="camera_depth_optical_frame"/>
+    <joint name="camera_depth_optical_joint" type="fixed">
+      <parent link="camera_depth_link"/>
+      <child link="camera_depth_optical_frame"/>
+      <origin xyz="0 0 0" rpy="-1.5708 0 -1.5708"/>
+    </joint>
+    <gazebo reference="camera_depth_link">
       <sensor name="d435_depth" type="depth">
+        <pose>0 0 0 0 0 -1.5708</pose>
         <update_rate>30.0</update_rate>
         <camera>
-          <horizontal_fov>1.39626</horizontal_fov>
+          <horizontal_fov>1.0472</horizontal_fov>
           <image>
             <width>640</width>
             <height>480</height>
-            <format>R8G8B8</format>
+            <format>DEPTH16</format>
           </image>
           <clip>
-            <near>0.1</near>
+            <near>0.01</near>
             <far>10.0</far>
           </clip>
         </camera>
-        <plugin name="d435_depth_plugin" filename="libgazebo_ros_camera.so">
+        <plugin name="depth_camera_controller" filename="libgazebo_ros_camera.so">
           <ros>
-            <namespace>/d435/depth</namespace>
+            <namespace>/camera_depth</namespace>
           </ros>
-          <camera_name>depth</camera_name>
+          <camera_name>depth_camera</camera_name>
           <image_topic_name>image_raw</image_topic_name>
           <camera_info_topic_name>camera_info</camera_info_topic_name>
           <frame_name>camera_depth_optical_frame</frame_name>
+          <output_encoding>32FC1</output_encoding>
         </plugin>
-        <plugin name="d435_pointcloud_plugin" filename="libgazebo_ros_point_cloud.so">
+        <plugin name="pointcloud_plugin" filename="libgazebo_ros_point_cloud.so">
           <ros>
-            <namespace>/d435</namespace>
+            <namespace>/camera_depth</namespace>
           </ros>
           <topic_name>points</topic_name>

File: MOBILE_MANIPULATOR/mobile_manipulator_description/urdf/mobile_manipulator.urdf.xacro (robot description, xacro)
@@ -40,7 +40,7 @@
   <xacro:intel_d435_camera/>
   <joint name="sliderto_camera" type="fixed">
-    <parent link="slider"/>
-    <child  link="camera_link"/>
-    <origin xyz="0 -0.5 0.1" rpy="0 0 -1.57"/>
+    <parent link="link_base"/>
+    <child  link="camera_link_base"/>
+    <origin xyz="-0.3 -0.3 0.85" rpy="0 0 0"/>
   </joint>
 </robot>

Commit message: Added lift withoiut doors and editted teh lift plugin

File: ALPHA_BOT/alphabot_description/urdf/alphabot.urdf.xacro (robot description, xacro)
@@ -47,5 +47,5 @@
         <parent link="base_footprint"/>
         <child link="link_base"/>
-        <origin xyz="-0.6 17.8 ${chassis_height/2 + traction_wheel_radius}" rpy="0 0 1.57" />
+        <origin xyz="0 0 ${chassis_height/2 + traction_wheel_radius}" rpy="0 0 1.57" />
     </joint>
     <link name="chassis_link">

File: MOBILE_MANIPULATOR/mobile_manipulator_description/urdf/mobile_manipulator.urdf.xacro (robot description, xacro)
@@ -38,4 +38,31 @@
     </gazebo>
   <xacro:include filename="$(find mobile_manipulator_description)/urdf/camera_module.urdf.xacro"/>
+  <link name="cylinder_link">
+  <visual>
+    <geometry>
+      <cylinder radius="0.01" length="0.71"/>
+    </geometry>
+    <material name="Grey">
+      <color rgba="0.7 0.7 0.7 1"/>
+    </material>
+  </visual>
+  <collision>
+    <geometry>
+      <cylinder radius="0.01" length="0.71"/>
+    </geometry>
+  </collision>
+  <inertial>
+    <mass value="0.5"/>
+    <inertia ixx="0.001" ixy="0" ixz="0" iyy="0.001" iyz="0" izz="0.001"/>
+  </inertial>
+</link>
+ <joint name="rod_to_camera" type="fixed">
+    <parent link="camera_link_base"/>
+    <child  link="cylinder_link"/>
+    <origin xyz="0.01 0 -0.36" rpy="0 0 0"/>
+  </joint>
+    <gazebo reference="cylinder_link">
+      <material>Gazebo/Grey</material>
+  </gazebo>
   <xacro:intel_d435_camera/>
   <joint name="sliderto_camera" type="fixed">

Commit message: Refactored pipleine and world file

File: ALPHA_BOT/alphabot_description/urdf/alphabot.urdf.xacro (robot description, xacro)
@@ -1,4 +1,4 @@
 <?xml version="1.0"?>
-<robot xmlns:xacro="http://www.ros.org/wiki/xacro" name="bcr_bot">
+<robot xmlns:xacro="http://www.ros.org/wiki/xacro" name="alpha_bot">
     <xacro:property name="chassis_mass" value="70"/>
     <xacro:property name="chassis_length" value="0.9"/>

File: ALPHA_BOT/alphabot_description/urdf/gazebo.xacro (robot description, xacro)
@@ -1,4 +1,4 @@
 <?xml version="1.0"?>
-<robot xmlns:xacro="http://www.ros.org/wiki/xacro" name="bcr_bot">
+<robot xmlns:xacro="http://www.ros.org/wiki/xacro" name="alpha_bot">
     <gazebo>
         <static>false</static>

File: ALPHA_BOT/alphabot_description/urdf/macros.xacro (robot description, xacro)
@@ -1,4 +1,4 @@
 <?xml version="1.0"?>
-<robot xmlns:xacro="http://www.ros.org/wiki/xacro" name="bcr_bot">
+<robot xmlns:xacro="http://www.ros.org/wiki/xacro" name="alpha_bot">
     <xacro:macro name="cylinder_inertia" params="m r h">
         <inertia ixx="${m * (3 * r * r + h * h) / 12}" ixy="0" ixz="0" iyy="${m * (3 * r * r + h * h) / 12}" iyz="0" izz="${m * r * r / 2}" />

File: ALPHA_BOT/alphabot_description/urdf/materials.xacro (robot description, xacro)
@@ -1,4 +1,4 @@
 <?xml version="1.0"?>
-<robot xmlns:xacro="http://www.ros.org/wiki/xacro" name="bcr_bot">
+<robot xmlns:xacro="http://www.ros.org/wiki/xacro" name="alpha_bot">
     <material name="black">
         <color rgba="0.0 0.0 0.0 1.0"/>

File: ALPHA_BOT/alphabot_navigation/urdf/alphabot.urdf.xacro (robot description, xacro)
@@ -1,4 +1,4 @@
 <?xml version="1.0"?>
-<robot xmlns:xacro="http://www.ros.org/wiki/xacro" name="bcr_bot">
+<robot xmlns:xacro="http://www.ros.org/wiki/xacro" name="alpha_bot">
     <xacro:property name="chassis_mass" value="70"/>
     <xacro:property name="chassis_length" value="0.9"/>

File: ALPHA_BOT/alphabot_navigation/urdf/gazebo.xacro (robot description, xacro)
@@ -1,4 +1,4 @@
 <?xml version="1.0"?>
-<robot xmlns:xacro="http://www.ros.org/wiki/xacro" name="bcr_bot">
+<robot xmlns:xacro="http://www.ros.org/wiki/xacro" name="alpha_bot">
     <gazebo>
         <static>false</static>

File: MOBILE_MANIPULATOR/mobile_manipulator_description/urdf/mobile_manipulator.urdf.xacro (robot description, xacro)
@@ -13,5 +13,5 @@
     <parent link="slider"/>
     <child  link="base_link"/>
-    <origin xyz="0 -0.33 0.06" rpy="0 0 -1.57"/>
+    <origin xyz="0 -0.37 0.06" rpy="0 0 0"/>
   </joint>
   <gazebo>
