Commit message: Enhance robot description and visualization by adding tool link and joint, updating URDF and SRDF files, and modifying target positions in JSON. Adjusted box spawner plugin parameters for improved functionality.

File: REALMAN_7DOF/rm_description/urdf/rm_75.urdf (robot description, URDF)
Before this commit: robot rm_75_description, 8 links, 7 joints
Links:
- added link tool0, mass 0.1; collision mesh filename=file://$(find rm_description)/meshes/rm_75_arm/object.stl scale=0.001 0.001 0.001; visual mesh filename=file://$(find rm_description)/meshes/rm_75_arm/object.stl scale=0.001 0.001 0.001
Joints:
- added joint joint_tool0: type fixed, parent Link7, child tool0, origin xyz=0 0 0.1 rpy=0 0 1.57

File: REALMAN_7DOF/rm_description/urdf/rm_75_gazebo.urdf (robot description, URDF)
Before this commit: robot rm_75_description, 8 links, 7 joints
Links:
- added link tool0, mass 0.001; collision mesh filename=file://$(find rm_description)/meshes/rm_75_arm/object.stl scale=0.001 0.001 0.001; visual mesh filename=file://$(find rm_description)/meshes/rm_75_arm/object.stl scale=0.001 0.001 0.001
Joints:
- added joint joint_tool0: type fixed, parent Link7, child tool0, origin xyz=0 0 0.1 rpy=0 0 1.57
